Commit message: parametrized arms

File: arena_robots/robots/rbrobout/urdf/rbrobout.urdf.xacro (robot description, xacro)
@@ -12,45 +12,10 @@
   <xacro:arg name="prefix" default="robot_"/>
   <xacro:arg name="sim_path" default=""/>
+  <xacro:arg name="gazebo_classic" default="false"/>
   <xacro:arg name="gazebo_ignition" default="true"/>
   <xacro:arg name="gazebo_controllers" default=""/>
-  <xacro:property name="front_laser_offset_x" value="0.8"/>
-  <xacro:property name="front_laser_offset_y" value="0.366"/>
-  <xacro:property name="front_laser_offset_z" value="-0.06"/>
-  <xacro:property name="rear_laser_offset_x" value="-0.8"/>
-  <xacro:property name="rear_laser_offset_y" value="-0.366"/>
-  <xacro:property name="rear_laser_offset_z" value="-0.06"/>
-  <xacro:property name="imu_offset_x" value="0.3"/>
-  <xacro:property name="imu_offset_y" value="-0.3"/>
-  <xacro:property name="imu_offset_z" value="0.0725"/>
   <xacro:rbrobout prefix="$(arg prefix)" gazebo_ignition="$(arg gazebo_ignition)"/>
-  <!-- IMU -->
-  <xacro:sensor_vectornav
-      frame_prefix="$(arg prefix)vectornav_"
-      parent="$(arg prefix)base_link"
-      node_namespace="$(arg namespace)"
-      gazebo_classic="false"
-      gazebo_ignition="$(arg gazebo_ignition)">
-      <origin xyz="${imu_offset_x} ${imu_offset_y} ${imu_offset_z}" rpy="0 0 0"/>
-  </xacro:sensor_vectornav>
-  <!-- 2d laser -->
-  <xacro:sensor_sick_microscan3
-      frame_prefix="$(arg prefix)front_laser_"
-      parent="$(arg prefix)base_link"
-      node_namespace="$(arg namespace)"
-      node_name="front_laser"
-      gazebo_classic="false"
-      gazebo_ignition="$(arg gazebo_ignition)">
-      <origin xyz="${front_laser_offset_x} ${front_laser_offset_y} ${front_laser_offset_z}" rpy="0 0 ${1/4*PI}"/>
-  </xacro:sensor_sick_microscan3>
-  <!-- 2d laser -->
-  <xacro:sensor_sick_microscan3
-      frame_prefix="$(arg prefix)rear_laser_"
-      parent="$(arg prefix)base_link"
-      node_namespace="$(arg namespace)"
-      node_name="rear_laser"
-      gazebo_classic="false"
-      gazebo_ignition="$(arg gazebo_ignition)">
-      <origin xyz="${rear_laser_offset_x} ${rear_laser_offset_y} ${rear_laser_offset_z}" rpy="0 0 ${-3/4*PI}"/>
-  </xacro:sensor_sick_microscan3>
+  <!-- SENSORS: migrated to the component catalog (assembly.yaml, Stage M); attached
+       by the per-robot wrapper xacro (catalog.render_wrapper_xacro), not here. -->
   <!-- ros2_control hardware block (always active; gz plugin loaded via rbrobout.gazebo) -->
   <xacro:rbrobout_base_hw_controller/>

File: arena_robots/robots/rbtheron/urdf/rbtheron.urdf.xacro (robot description, xacro)
@@ -27,67 +27,6 @@
 	<!-- Here we create the robot using the xacro:macro imported at the beggining of this file -->
 	<xacro:rbtheron prefix="$(arg prefix)" hq="${hq}"/>
-	<!-- SENSORS -->
-    <xacro:property name="imu_offset_x" value="-0.1975"/>
-    <xacro:property name="imu_offset_y" value="0.0"/>
-    <xacro:property name="imu_offset_z" value="0.1598"/>
-	<xacro:property name="front_rgbd_camera_offset_x" value="0.3045"/>
-	<xacro:property name="front_rgbd_camera_offset_y" value="0.0"/>
-	<xacro:property name="front_rgbd_camera_offset_z" value="0.1898"/>
-	<xacro:property name="rear_rgbd_camera_offset_x" value="-0.3045"/>
-	<xacro:property name="rear_rgbd_camera_offset_y" value="0.0"/>
-	<xacro:property name="rear_rgbd_camera_offset_z" value="0.1158"/>
-	<xacro:property name="front_laser_offset_x" value="0.2675"/>
-	<xacro:property name="front_laser_offset_y" value="-0.215"/>
-	<xacro:property name="front_laser_offset_z" value="0.1613"/>
-	<xacro:property name="rear_laser_offset_x" value="-0.2675"/>
-	<xacro:property name="rear_laser_offset_y" value="0.215"/>
-	<xacro:property name="rear_laser_offset_z" value="0.1613"/>
-	<!-- IMU -->
-    <xacro:sensor_vectornav
-        frame_prefix="$(arg prefix)vectornav_"
-        parent="$(arg prefix)base_link"
-        node_namespace="$(arg namespace)"
-        gazebo_classic="$(arg gazebo_classic)"
-        gazebo_ignition="$(arg gazebo_ignition)">
-        <origin xyz="${imu_offset_x} ${imu_offset_y} ${imu_offset_z}" rpy="0 0 0"/>
-    </xacro:sensor_vectornav>
-	<!-- 2D LASER -->
-    <xacro:sensor_hokuyo_ust20lx
-        frame_prefix="$(arg prefix)front_laser_"
-        parent="$(arg prefix)base_link"
-        node_namespace="$(arg namespace)"
-        node_name="front_laser"
-        gazebo_classic="$(arg gazebo_classic)"
-        gazebo_ignition="$(arg gazebo_ignition)">
-        <origin xyz="${front_laser_offset_x} ${front_laser_offset_y} ${front_laser_offset_z}" rpy="0 ${-PI} ${3/4*PI}"/>
-    </xacro:sensor_hokuyo_ust20lx>
-    <xacro:sensor_hokuyo_ust20lx
-        frame_prefix="$(arg prefix)rear_laser_"
-        parent="$(arg prefix)base_link"
-        node_namespace="$(arg namespace)"
-        node_name="rear_laser"
-        gazebo_classic="$(arg gazebo_classic)"
-        gazebo_ignition="$(arg gazebo_ignition)">
-        <origin xyz="${rear_laser_offset_x} ${rear_laser_offset_y} ${rear_laser_offset_z}" rpy="0 ${-PI} ${-1/4*PI}"/>
-    </xacro:sensor_hokuyo_ust20lx>
-  	<!-- CAMERAS -->
-    <xacro:sensor_intel_realsense_d435
-        frame_prefix="$(arg prefix)front_rgbd_camera_"
-        parent="$(arg prefix)base_link"
-        node_namespace="$(arg namespace)"
-        node_name="front_camera"
-        gazebo_classic="$(arg gazebo_classic)"
-        gazebo_ignition="$(arg gazebo_ignition)">
-        <origin xyz="${front_rgbd_camera_offset_x} ${front_rgbd_camera_offset_y} ${front_rgbd_camera_offset_z}" rpy="0 0 0"/>
-    </xacro:sensor_intel_realsense_d435>
-    <xacro:sensor_intel_realsense_d435
-        frame_prefix="$(arg prefix)rear_rgbd_camera_"
-        parent="$(arg prefix)base_link"
-        node_namespace="$(arg namespace)"
-        node_name="rear_camera"
-        gazebo_classic="$(arg gazebo_classic)"
-        gazebo_ignition="$(arg gazebo_ignition)">
-        <origin xyz="${rear_rgbd_camera_offset_x} ${rear_rgbd_camera_offset_y} ${rear_rgbd_camera_offset_z}" rpy="0 0 ${PI}"/>
-    </xacro:sensor_intel_realsense_d435>
+	<!-- SENSORS: migrated to the component catalog (assembly.yaml, Stage M); attached
+	     by the per-robot wrapper xacro (catalog.render_wrapper_xacro), not here. -->
 	<!-- Controllers -->
 	<xacro:if value="$(arg gazebo_classic)">

File: arena_robots/robots/rbvogui/urdf/rbvogui.urdf.xacro (robot description, xacro)
@@ -19,55 +19,13 @@
 	<xacro:arg name="sim_path" default=""/>
 	<xacro:arg name="gazebo_controllers" default=""/>
+	<xacro:arg name="gazebo_classic" default="false"/>
+	<xacro:arg name="gazebo_ignition" default="true"/>
+	<xacro:arg name="generate_ros2_control_tag" default="true"/>
     <xacro:rbvogui prefix="$(arg prefix)" hq="${hq}"/>
-    <!-- SENSORS see robotnik_sensors for the specific configuration -->
-    <!-- IMU -->
-    <xacro:sensor_vectornav
-        frame_prefix="$(arg prefix)vectornav_"
-        parent="$(arg prefix)chassis_link"
-        node_namespace="$(arg namespace)"
-        gazebo_classic="false"
-        gazebo_ignition="true">
-        <origin xyz="0.3 -0.3 0.0725" rpy="0 0 0"/>
-    </xacro:sensor_vectornav>
-    <!-- Front Camera -->
-    <xacro:sensor_intel_realsense_d435
-        frame_prefix="$(arg prefix)front_rgbd_camera_"
-        parent="$(arg prefix)base_link"
-        node_namespace="$(arg namespace)"
-        node_name="front_camera"
-        gazebo_classic="false"
-        gazebo_ignition="true">
-        <origin xyz="0.46462 0.0 0.18258" rpy="0 0 0"/>
-    </xacro:sensor_intel_realsense_d435>
-    <!-- Rear Camera -->
-    <xacro:sensor_intel_realsense_d435
-        frame_prefix="$(arg prefix)rear_rgbd_camera_"
-        parent="$(arg prefix)base_link"
-        node_namespace="$(arg namespace)"
-        node_name="rear_camera"
-        gazebo_classic="false"
-        gazebo_ignition="true">
-        <origin xyz="-0.503 0.0 0.29" rpy="0 0 -${PI}"/>
-    </xacro:sensor_intel_realsense_d435>
-    <!-- 2d laser -->
-    <xacro:sensor_sick_s300
-        frame_prefix="$(arg prefix)front_laser_"
-        parent="$(arg prefix)chassis_link"
-        node_namespace="$(arg namespace)"
-        node_name="front_laser"
-        gazebo_classic="false"
-        gazebo_ignition="true">
-        <origin xyz="0.53 0.33 0.1145" rpy="${PI} 0 ${PI/4}"/>
-    </xacro:sensor_sick_s300>
-    <xacro:sensor_sick_s300
-        frame_prefix="$(arg prefix)rear_laser_"
-        parent="$(arg prefix)chassis_link"
-        node_namespace="$(arg namespace)"
-        node_name="rear_laser"
-        gazebo_classic="false"
-        gazebo_ignition="true">
-        <origin xyz="-0.53 -0.33 0.1145" rpy="${PI} 0 ${-PI*3/4}"/>
-    </xacro:sensor_sick_s300>
+    <!-- SENSORS: migrated to the component catalog (assembly.yaml, Stage M); attached
+         by the per-robot wrapper xacro (catalog.render_wrapper_xacro), not here. -->
     <!-- ros2_control block (gz_ros2_control/GazeboSimSystem) and PosePublisher loaded via rbvogui.gazebo -->
-    <xacro:rbvogui_base_hw_controller/>
+    <xacro:if value="$(arg generate_ros2_control_tag)">
+        <xacro:rbvogui_base_hw_controller/>
+    </xacro:if>
 </robot>
