Commit message: migrate mpo700, rskomnidirectional, ridgeback

File: arena_robots/robots/mpo700/urdf/mpo700.urdf.xacro (robot description, xacro)
@@ -2,6 +2,9 @@
 <robot name="mpo700" xmlns:xacro="http://www.ros.org/wiki/xacro">
   <xacro:arg name="namespace" default=""/>
+  <xacro:arg name="prefix" default=""/>
   <xacro:arg name="sim_path" default=""/>
   <xacro:arg name="gazebo_controllers" default=""/>
+  <xacro:arg name="gazebo_classic" default="false"/>
+  <xacro:arg name="gazebo_ignition" default="true"/>
   <xacro:property name="ODM_joint_type" value="continuous"/>
   <xacro:include filename="$(find arena_robots)/robots/mpo700/urdf/xacros/mpo_700_body.urdf.xacro"/>
@@ -9,24 +12,7 @@
   <xacro:include filename="$(find arena_robots)/robots/mpo700/urdf/mpo700.gazebo"/>
   <xacro:include filename="$(find arena_robots)/robots/rbvogui/urdf/utils/inertia.urdf.xacro"/>
-  <xacro:include filename="$(find arena_robots)/robots/rbvogui/urdf/2d_lidar/sick_s300.urdf.xacro"/>
   <xacro:mpo_700_body/>
-  <xacro:sensor_sick_s300
-    frame_prefix="front_laser_"
-    parent="base_footprint"
-    node_namespace="$(arg namespace)"
-    node_name="front_laser"
-    gazebo_classic="false"
-    gazebo_ignition="true">
-    <origin xyz="0.338 0.288 0.223" rpy="3.14 0 0.79"/>
-  </xacro:sensor_sick_s300>
-  <xacro:sensor_sick_s300
-    frame_prefix="rear_laser_"
-    parent="base_footprint"
-    node_namespace="$(arg namespace)"
-    node_name="rear_laser"
-    gazebo_classic="false"
-    gazebo_ignition="true">
-    <origin xyz="-0.338 -0.288 0.223" rpy="3.14 0 3.93"/>
-  </xacro:sensor_sick_s300>
+  <!-- SENSORS: migrated to the component catalog (assembly.yaml, Stage M); attached
+       by the per-robot wrapper xacro (catalog.render_wrapper_xacro), not here. -->
   <xacro:mpo700_base_hw_controller/>
 </robot>

File: arena_robots/robots/ridgeback/urdf/ridgeback.urdf.xacro (robot description, xacro)
@@ -288,9 +288,10 @@
   <xacro:include filename="$(find arena_robots)/robots/ridgeback/urdf/base_hw/ridgeback.ros2_control.urdf"/>
   <xacro:include filename="$(find arena_robots)/robots/ridgeback/urdf/ridgeback.gazebo" />
-  <!-- gz-sim sensors; imu_link is already used for the kinematic frame -->
-  <xacro:arg name="sim_path" default=""/>
-  <xacro:include filename="$(find arena_robots)/config/urdf/sensors/default.xacro"/>
-  <xacro:arena_default_lidar parent_link="base_link"/>
-  <xacro:arena_default_imu parent_link="base_link" frame="imu_sensor_link"/>
+  <!-- SENSORS: migrated to the component catalog (assembly.yaml, Stage M); attached
+       by the per-robot wrapper xacro (catalog.render_wrapper_xacro), not here. -->
+  <xacro:arg name="namespace" default=""/>
+  <xacro:arg name="prefix" default=""/>
+  <xacro:arg name="gazebo_classic" default="false"/>
+  <xacro:arg name="gazebo_ignition" default="true"/>
   <!-- Optional standard accessories, including their simulation data. The rendering
        of these into the final description is controlled by optenv variables, which

File: arena_robots/tests/golden/rskomnidirectional_premigration.urdf (robot description, URDF)
Before this commit: robot urdf, 114 links, 113 joints
Links:
- added link imu_link
- added link lidar
Joints:
- added joint imu_link_joint: type fixed, parent base, child imu_link, origin xyz=0 0 0 rpy=0 0 0
- added joint lidar_joint: type fixed, parent base, child lidar, origin xyz=0 0 0.3 rpy=0 0 0
