Commit message: migrate rbkairos

File: arena_robots/robots/rbkairos/urdf/rbkairos.urdf.xacro (robot description, xacro)
@@ -16,55 +16,5 @@
   <xacro:arg name="gazebo_controllers" default=""/>
   <xacro:arg name="sim_path" default=""/>
-  <xacro:property name="front_laser_offset_x" value="0.42109"/>
-  <xacro:property name="front_laser_offset_y" value="-0.32737"/>
-  <xacro:property name="front_laser_offset_z" value="0.16037"/>
-  <xacro:property name="rear_laser_offset_x" value="-0.42109"/>
-  <xacro:property name="rear_laser_offset_y" value="0.32737"/>
-  <xacro:property name="rear_laser_offset_z" value="0.16037"/>
-  <xacro:property name="imu_offset_x" value="0.127"/>
-  <xacro:property name="imu_offset_y" value="-0.129"/>
-  <xacro:property name="imu_offset_z" value="0.212"/>
-  <xacro:property name="front_rgbd_camera_offset_x" value="0.35850"/>
-  <xacro:property name="front_rgbd_camera_offset_y" value="0.0"/>
-  <xacro:property name="front_rgbd_camera_offset_z" value="0.25062"/>
   <xacro:rbkairos prefix="$(arg prefix)" gazebo_classic="$(arg gazebo_classic)" gazebo_ignition="$(arg gazebo_ignition)"/>
-  <!-- IMU -->
-    <xacro:sensor_vectornav
-        frame_prefix="$(arg prefix)vectornav_"
-        parent="$(arg prefix)base_link"
-        node_namespace="$(arg namespace)"
-        gazebo_classic="$(arg gazebo_classic)"
-        gazebo_ignition="$(arg gazebo_ignition)">
-        <origin xyz="${imu_offset_x} ${imu_offset_y} ${imu_offset_z}" rpy="0 0 0"/>
-    </xacro:sensor_vectornav>
-  <!-- SENSORS -->
-    <xacro:sensor_sick_s300
-        frame_prefix="$(arg prefix)front_laser_"
-        parent="$(arg prefix)base_link"
-        node_namespace="$(arg namespace)"
-        node_name="front_laser"
-        gazebo_classic="$(arg gazebo_classic)"
-        gazebo_ignition="$(arg gazebo_ignition)">
-        <origin xyz="${front_laser_offset_x} ${front_laser_offset_y} ${front_laser_offset_z}" rpy="0 ${-PI} ${3/4*PI}"/>
-    </xacro:sensor_sick_s300>
-    <xacro:sensor_sick_s300
-        frame_prefix="$(arg prefix)rear_laser_"
-        parent="$(arg prefix)base_link"
-        node_namespace="$(arg namespace)"
-        node_name="rear_laser"
-        gazebo_classic="$(arg gazebo_classic)"
-        gazebo_ignition="$(arg gazebo_ignition)">
-        <origin xyz="${rear_laser_offset_x} ${rear_laser_offset_y} ${rear_laser_offset_z}" rpy="0 ${-PI} ${-1/4*PI}"/>
-    </xacro:sensor_sick_s300>
-  <!-- CAMERA -->
-    <xacro:sensor_intel_realsense_d435
-        frame_prefix="$(arg prefix)front_rgbd_camera_"
-        parent="$(arg prefix)base_link"
-        node_namespace="$(arg namespace)"
-        node_name="front_camera"
-        gazebo_classic="$(arg gazebo_classic)"
-        gazebo_ignition="$(arg gazebo_ignition)">
-        <origin xyz="${front_rgbd_camera_offset_x} ${front_rgbd_camera_offset_y} ${front_rgbd_camera_offset_z}" rpy="0 0 0"/>
-    </xacro:sensor_intel_realsense_d435>
   <!-- Controllers -->
   <xacro:if value="$(arg gazebo_classic)">
