Commit message: migrate boxer, a1, go1

File: arena_robots/robots/a1/urdf/a1.urdf.xacro (robot description, xacro)
@@ -5,9 +5,9 @@
   <xacro:arg name="namespace" default="" />
   <xacro:arg name="gazebo_controllers" default="" />
+  <xacro:arg name="gazebo_classic" default="false" />
+  <xacro:arg name="gazebo_ignition" default="true" />
   <xacro:include filename="$(find arena_robots)/robots/a1/urdf/include/const.xacro" />
   <xacro:include filename="$(find arena_robots)/robots/a1/urdf/include/materials.xacro" />
   <xacro:include filename="$(find arena_robots)/robots/a1/urdf/include/leg.xacro" />
-  <xacro:include filename="$(find arena_robots)/robots/a1/urdf/include/depthcamera.xacro" />
-  <xacro:include filename="$(find arena_robots)/urdf/gz_lidar.xacro" />
   <link name="base">
     <visual>
@@ -70,27 +70,4 @@
     <origin rpy="0 0 0" xyz="${-leg_offset_x} ${leg_offset_y} 0"/>
   </xacro:leg>
-  <xacro:a1_depth_camera name="face">
-    <origin rpy="0 0 0" xyz="0.271 0.0125 0.0167"/>
-  </xacro:a1_depth_camera>
-  <joint name="lidar_joint" type="fixed">
-    <parent link="trunk" />
-    <child link="lidar" />
-    <origin xyz="0 0 0.10" rpy="0 0 0" />
-  </joint>
-  <link name="lidar">
-    <visual>
-      <origin xyz="0 0 0" rpy="0 0 0" />
-      <geometry>
-        <cylinder length="0.05" radius="0.04" />
-      </geometry>
-      <material name="black" />
-    </visual>
-    <inertial>
-      <mass value="1e-5" />
-      <origin xyz="0 0 0" rpy="0 0 0" />
-      <inertia ixx="1e-6" ixy="0" ixz="0" iyy="1e-6" iyz="0" izz="1e-6" />
-    </inertial>
-  </link>
-  <xacro:gz_lidar frame="lidar" />
   <xacro:include filename="$(find arena_robots)/robots/a1/urdf/base_hw/a1.ros2_control.urdf" />
   <xacro:a1_base_hw_controller/>

File: arena_robots/robots/boxer/urdf/boxer.urdf.xacro (robot description, xacro)
@@ -118,11 +118,12 @@
   <!-- Include sub files -->
   <xacro:arg name="sim_path" default=""/>
+  <xacro:arg name="namespace" default=""/>
+  <xacro:arg name="prefix" default=""/>
+  <xacro:arg name="gazebo_classic" default="false"/>
+  <xacro:arg name="gazebo_ignition" default="true"/>
   <xacro:include filename="$(find arena_robots)/robots/boxer/urdf/include/sensors.urdf.xacro" />
   <xacro:include filename="$(find arena_robots)/robots/boxer/urdf/include/wheels_and_casters.urdf.xacro" />
   <xacro:include filename="$(find arena_robots)/robots/boxer/urdf/base_hw/boxer.ros2_control.urdf" />
   <xacro:include filename="$(find arena_robots)/robots/boxer/urdf/boxer.gazebo" />
-  <!-- gz-sim IMU sensor; imu_link is already used for kinematic placement -->
-  <xacro:include filename="$(find arena_robots)/config/urdf/sensors/default.xacro"/>
-  <xacro:arena_default_imu parent_link="base_link" frame="imu_sensor_link"/>
   <xacro:boxer_base_hw_controller/>
   <!-- User extensions -->

File: arena_robots/robots/boxer/urdf/include/sensors.urdf.xacro (robot description, xacro)
@@ -72,105 +72,4 @@
     </sensor>
   </gazebo>
-  <!-- Front safety sensor -->
-  <link name="front_laser">
-    <visual>
-      <geometry>
-        <mesh filename="package://arena_robots/robots/boxer/meshes/hokuyo_uam_05lp.stl" scale="0.001 0.001 0.001" />
-      </geometry>
-      <origin xyz="0 0 0" rpy="0 0 0" />
-      <material name="Boxer_Black" />
-    </visual>
-  </link>
-  <joint name="front_laser_joint" type="fixed">
-    <parent link="chassis_link" />
-    <child link="front_laser" />
-    <origin xyz="0.3062 0 0.1614" rpy="0 0 0" />
-  </joint>
-  <gazebo reference="front_laser">
-    <material>Gazebo/Black</material>
-    <turnGravityOff>true</turnGravityOff>
-    <sensor type="gpu_lidar" name="front_laser">
-      <gz_frame_id>$(arg sim_path)/front_laser</gz_frame_id>
-      <pose>0 0 0 0 0 0</pose>
-      <visualize>false</visualize>
-      <update_rate>33</update_rate>
-      <ray>
-        <scan>
-          <horizontal>
-            <samples>720</samples>
-            <resolution>1</resolution>
-            <min_angle>-2.35619449019</min_angle>
-            <max_angle>2.35619449019</max_angle>
-          </horizontal>
-        </scan>
-        <range>
-          <min>0.5</min>
-          <max>20</max>
-          <resolution>0.01</resolution>
-        </range>
-        <noise>
-          <type>gaussian</type>
-          <mean>0.0</mean>
-          <stddev>0.001</stddev>
-        </noise>
-      </ray>
-      <plugin name="gazebo_ros_laser" filename="libgazebo_ros_laser.so">
-        <topicName>front/scan</topicName>
-        <frameName>front_laser</frameName>
-        <robotNamespace>/</robotNamespace>
-      </plugin>
-    </sensor>
-  </gazebo>
-  <!-- Internal rear safety laser -->
-  <link name="rear_sensor">
-    <visual>
-      <geometry>
-        <mesh filename="package://arena_robots/robots/boxer/meshes/rear_sensor.stl" scale="0.001 0.001 0.001" />
-      </geometry>
-      <origin xyz="0 0 0" rpy="0 0 ${pi}" />
-      <material name="Boxer_Black" />
-    </visual>
-  </link>
-  <joint name="rear_sensor_joint" type="fixed">
-    <parent link="chassis_link" />
-    <child link="rear_sensor" />
-    <origin xyz="-0.3404 0.0241 0.0779" rpy="0 -0.0698131700798 ${pi}" />
-  </joint>
-  <!-- TODO look up the actual specs for this sensor; range, FoV, samples is a complete guess right now -->
-  <gazebo reference="rear_sensor">
-    <material>Gazebo/Black</material>
-    <turnGravityOff>true</turnGravityOff>
-    <sensor type="gpu_lidar" name="rear_laser">
-      <gz_frame_id>$(arg sim_path)/rear_sensor</gz_frame_id>
-      <pose>0 0 0 0 0 0</pose>
-      <visualize>false</visualize>
-      <update_rate>33</update_rate>
-      <ray>
-        <scan>
-          <horizontal>
-            <samples>90</samples>
-            <resolution>1</resolution>
-            <min_angle>0.785398163397</min_angle>
-            <max_angle>-0.785398163397</max_angle>
-          </horizontal>
-        </scan>
-        <range>
-          <min>0.1</min>
-          <max>5</max>
-          <resolution>0.01</resolution>
-        </range>
-        <noise>
-          <type>gaussian</type>
-          <mean>0.0</mean>
-          <stddev>0.001</stddev>
-        </noise>
-      </ray>
-      <plugin name="gazebo_ros_laser" filename="libgazebo_ros_laser.so">
-        <topicName>rear/scan</topicName>
-        <frameName>rear_sensor</frameName>
-        <robotNamespace>/</robotNamespace>
-      </plugin>
-    </sensor>
-  </gazebo>
   <!-- Cart sensor -->
   <link name="cart_sensor"/>

File: arena_robots/robots/go1/urdf/go1.urdf.xacro (robot description, xacro)
@@ -5,9 +5,9 @@
   <xacro:arg name="namespace" default="" />
   <xacro:arg name="gazebo_controllers" default="" />
+  <xacro:arg name="gazebo_classic" default="false" />
+  <xacro:arg name="gazebo_ignition" default="true" />
   <xacro:include filename="$(find arena_robots)/robots/go1/urdf/include/const.xacro" />
   <xacro:include filename="$(find arena_robots)/robots/go1/urdf/include/materials.xacro" />
   <xacro:include filename="$(find arena_robots)/robots/go1/urdf/include/leg.xacro" />
-  <xacro:include filename="$(find arena_robots)/robots/go1/urdf/include/depthcamera.xacro" />
-  <xacro:include filename="$(find arena_robots)/urdf/gz_lidar.xacro" />
   <link name="base">
     <visual>
@@ -70,45 +70,4 @@
     <origin rpy="0 0 0" xyz="${-leg_offset_x} ${leg_offset_y} 0"/>
   </xacro:leg>
-  <!-- Go1 ships 5 depth/AI cameras (face, chin, left, right, rearDown). Only the
-       front (face) camera is active for now; each rgbd pass is render-heavy, so the
-       other 4 are commented out until needed (re-enable alongside mappings.yaml +
-       model_params.yaml). Drop resolution in depthcamera.xacro if RTF suffers. -->
-  <xacro:go1_depth_camera camID="1" name="face">
-    <origin rpy="${PI} 0 0" xyz="0.2785 0.0125 0.0167"/>
-  </xacro:go1_depth_camera>
-  <!--
-  <xacro:go1_depth_camera camID="2" name="chin">
-    <origin rpy="${PI} ${PI/2} 0" xyz="0.2522 0.0125 -0.0436"/>
-  </xacro:go1_depth_camera>
-  <xacro:go1_depth_camera camID="3" name="left">
-    <origin rpy="${PI} 0.2618 ${PI/2}" xyz="-0.066 0.082 -0.0176"/>
-  </xacro:go1_depth_camera>
-  <xacro:go1_depth_camera camID="4" name="right">
-    <origin rpy="${PI} 0.2618 ${-PI/2}" xyz="-0.041 -0.082 -0.0176"/>
-  </xacro:go1_depth_camera>
-  <xacro:go1_depth_camera camID="5" name="rearDown">
-    <origin rpy="${PI} ${PI/2} 0" xyz="-0.0825 0.0125 -0.04365"/>
-  </xacro:go1_depth_camera>
-  -->
-  <joint name="lidar_joint" type="fixed">
-    <parent link="trunk" />
-    <child link="lidar" />
-    <origin xyz="0 0 0.10" rpy="0 0 0" />
-  </joint>
-  <link name="lidar">
-    <visual>
-      <origin xyz="0 0 0" rpy="0 0 0" />
-      <geometry>
-        <cylinder length="0.05" radius="0.04" />
-      </geometry>
-      <material name="grey" />
-    </visual>
-    <inertial>
-      <mass value="1e-5" />
-      <origin xyz="0 0 0" rpy="0 0 0" />
-      <inertia ixx="1e-6" ixy="0" ixz="0" iyy="1e-6" iyz="0" izz="1e-6" />
-    </inertial>
-  </link>
-  <xacro:gz_lidar frame="lidar" />
   <xacro:include filename="$(find arena_robots)/robots/go1/urdf/base_hw/go1.ros2_control.urdf" />
   <xacro:go1_base_hw_controller/>
