Commit message: wire prefix through a1 and go1

File: arena_robots/robots/a1/urdf/a1.urdf.xacro (robot description, xacro)
@@ -10,5 +10,5 @@
   <xacro:include filename="$(find arena_robots)/robots/a1/urdf/include/materials.xacro" />
   <xacro:include filename="$(find arena_robots)/robots/a1/urdf/include/leg.xacro" />
-  <link name="base">
+  <link name="$(arg prefix)base">
     <visual>
       <origin rpy="0 0 0" xyz="0 0 0"/>
@@ -18,10 +18,10 @@
     </visual>
   </link>
-  <joint name="floating_base" type="fixed">
+  <joint name="$(arg prefix)floating_base" type="fixed">
     <origin rpy="0 0 0" xyz="0 0 0"/>
-    <parent link="base"/>
-    <child link="trunk"/>
+    <parent link="$(arg prefix)base"/>
+    <child link="$(arg prefix)trunk"/>
   </joint>
-  <link name="trunk">
+  <link name="$(arg prefix)trunk">
     <visual>
       <origin rpy="0 0 0" xyz="0 0 0"/>
@@ -46,10 +46,10 @@
     </inertial>
   </link>
-  <joint name="imu_joint" type="fixed">
-    <parent link="trunk"/>
-    <child link="imu_link"/>
+  <joint name="$(arg prefix)imu_joint" type="fixed">
+    <parent link="$(arg prefix)trunk"/>
+    <child link="$(arg prefix)imu_link"/>
     <origin rpy="0 0 0" xyz="0 0 0"/>
   </joint>
-  <link name="imu_link">
+  <link name="$(arg prefix)imu_link">
     <inertial>
       <mass value="0.001"/>
@@ -58,18 +58,18 @@
     </inertial>
   </link>
-  <xacro:leg name="FR" mirror="-1" mirror_dae="False" front_hind="1" front_hind_dae="True">
+  <xacro:leg name="FR" prefix="$(arg prefix)" mirror="-1" mirror_dae="False" front_hind="1" front_hind_dae="True">
     <origin rpy="0 0 0" xyz="${leg_offset_x} ${-leg_offset_y} 0"/>
   </xacro:leg>
-  <xacro:leg name="FL" mirror="1" mirror_dae="True" front_hind="1" front_hind_dae="True">
+  <xacro:leg name="FL" prefix="$(arg prefix)" mirror="1" mirror_dae="True" front_hind="1" front_hind_dae="True">
     <origin rpy="0 0 0" xyz="${leg_offset_x} ${leg_offset_y} 0"/>
   </xacro:leg>
-  <xacro:leg name="RR" mirror="-1" mirror_dae="False" front_hind="-1" front_hind_dae="False">
+  <xacro:leg name="RR" prefix="$(arg prefix)" mirror="-1" mirror_dae="False" front_hind="-1" front_hind_dae="False">
     <origin rpy="0 0 0" xyz="${-leg_offset_x} ${-leg_offset_y} 0"/>
   </xacro:leg>
-  <xacro:leg name="RL" mirror="1" mirror_dae="True" front_hind="-1" front_hind_dae="False">
+  <xacro:leg name="RL" prefix="$(arg prefix)" mirror="1" mirror_dae="True" front_hind="-1" front_hind_dae="False">
     <origin rpy="0 0 0" xyz="${-leg_offset_x} ${leg_offset_y} 0"/>
   </xacro:leg>
   <xacro:include filename="$(find arena_robots)/robots/a1/urdf/base_hw/a1.ros2_control.urdf" />
-  <xacro:a1_base_hw_controller/>
+  <xacro:a1_base_hw_controller prefix="$(arg prefix)"/>
   <gazebo>
     <plugin filename="libgz_ros2_control-system.so" name="gz_ros2_control::GazeboSimROS2ControlPlugin">
@@ -92,6 +92,6 @@
   </gazebo>
   <!-- Foot traction: legged stance needs high friction at the contact spheres. -->
-  <xacro:macro name="foot_friction" params="leg">
-    <gazebo reference="${leg}_foot">
+  <xacro:macro name="foot_friction" params="leg prefix">
+    <gazebo reference="${prefix}${leg}_foot">
       <mu1>0.8</mu1>
       <mu2>0.8</mu2>
@@ -100,7 +100,7 @@
     </gazebo>
   </xacro:macro>
-  <xacro:foot_friction leg="FL"/>
-  <xacro:foot_friction leg="FR"/>
-  <xacro:foot_friction leg="RL"/>
-  <xacro:foot_friction leg="RR"/>
+  <xacro:foot_friction leg="FL" prefix="$(arg prefix)"/>
+  <xacro:foot_friction leg="FR" prefix="$(arg prefix)"/>
+  <xacro:foot_friction leg="RL" prefix="$(arg prefix)"/>
+  <xacro:foot_friction leg="RR" prefix="$(arg prefix)"/>
 </robot>

File: arena_robots/robots/a1/urdf/include/depthcamera.xacro (robot description, xacro)
@@ -2,11 +2,11 @@
 <robot xmlns:xacro="http://www.ros.org/wiki/xacro">
   <xacro:include filename="$(find arena_robots)/urdf/gz_rgbd_camera.xacro"/>
-  <xacro:macro name="a1_depth_camera" params="name *origin">
-    <joint name="camera_joint_${name}" type="fixed">
+  <xacro:macro name="a1_depth_camera" params="name prefix:='' *origin">
+    <joint name="${prefix}camera_joint_${name}" type="fixed">
       <xacro:insert_block name="origin"/>
-      <parent link="trunk"/>
-      <child link="camera_${name}"/>
+      <parent link="${prefix}trunk"/>
+      <child link="${prefix}camera_${name}"/>
     </joint>
-    <link name="camera_${name}">
+    <link name="${prefix}camera_${name}">
       <visual>
         <origin xyz="0 0 0" rpy="0 0 0"/>
@@ -22,11 +22,11 @@
       </inertial>
     </link>
-    <joint name="camera_optical_joint_${name}" type="fixed">
+    <joint name="${prefix}camera_optical_joint_${name}" type="fixed">
       <origin xyz="0 0 0" rpy="${-pi/2} 0 ${-pi/2}"/>
-      <parent link="camera_${name}"/>
-      <child link="camera_optical_${name}"/>
+      <parent link="${prefix}camera_${name}"/>
+      <child link="${prefix}camera_optical_${name}"/>
     </joint>
-    <link name="camera_optical_${name}"/>
-    <xacro:gz_rgbd_camera frame="camera_${name}" sensor_name="camera_${name}"
+    <link name="${prefix}camera_optical_${name}"/>
+    <xacro:gz_rgbd_camera frame="${prefix}camera_${name}" sensor_name="${prefix}camera_${name}"
                           fov="2.094" width="640" height="480" near="0.05" far="8.0"
                           update_rate="15"/>

File: arena_robots/robots/a1/urdf/include/leg.xacro (robot description, xacro)
@@ -1,9 +1,9 @@
 <?xml version="1.0"?>
 <robot xmlns:xacro="http://www.ros.org/wiki/xacro">
-    <xacro:macro name="leg" params="name mirror mirror_dae front_hind front_hind_dae *origin">
-        <joint name="${name}_hip_joint" type="revolute">
+    <xacro:macro name="leg" params="name prefix mirror mirror_dae front_hind front_hind_dae *origin">
+        <joint name="${prefix}${name}_hip_joint" type="revolute">
             <xacro:insert_block name="origin"/>
-            <parent link="trunk"/>
-            <child link="${name}_hip"/>
+            <parent link="${prefix}trunk"/>
+            <child link="${prefix}${name}_hip"/>
             <axis xyz="1 0 0"/>
             <dynamics damping="${damping}" friction="${friction}"/>
@@ -15,5 +15,5 @@
             </xacro:if>
         </joint>
-        <link name="${name}_hip">
+        <link name="${prefix}${name}_hip">
             <visual>
                 <xacro:if value="${(mirror_dae == True) and (front_hind_dae == True)}">
@@ -49,11 +49,11 @@
             </inertial>
         </link>
-        <joint name="${name}_hip_fixed" type="fixed">
+        <joint name="${prefix}${name}_hip_fixed" type="fixed">
             <origin rpy="0 0 0" xyz="0 ${(thigh_shoulder_length/2.0+hip_offset)*mirror} 0"/>
-            <parent link="${name}_hip"/>
-            <child link="${name}_thigh_shoulder"/>
+            <parent link="${prefix}${name}_hip"/>
+            <child link="${prefix}${name}_thigh_shoulder"/>
         </joint>
         <!-- this link is only for collision -->
-        <link name="${name}_thigh_shoulder">
+        <link name="${prefix}${name}_thigh_shoulder">
             <collision>
                 <origin rpy="${PI/2.0} 0 0" xyz="0 0 0"/>
@@ -63,13 +63,13 @@
             </collision>
         </link>
-        <joint name="${name}_thigh_joint" type="revolute">
+        <joint name="${prefix}${name}_thigh_joint" type="revolute">
             <origin rpy="0 0 0" xyz="0 ${thigh_offset*mirror} 0"/>
-            <parent link="${name}_hip"/>
-            <child link="${name}_thigh"/>
+            <parent link="${prefix}${name}_hip"/>
+            <child link="${prefix}${name}_thigh"/>
             <axis xyz="0 1 0"/>
             <dynamics damping="${damping}" friction="${friction}"/>
             <limit effort="${thigh_torque_max}" velocity="${thigh_velocity_max}" lower="${thigh_min*PI/180.0}" upper="${thigh_max*PI/180.0}"/>
         </joint>
-        <link name="${name}_thigh">
+        <link name="${prefix}${name}_thigh">
             <visual>
                 <origin rpy="0 0 0" xyz="0 0 0"/>
@@ -99,13 +99,13 @@
             </inertial>
         </link>
-        <joint name="${name}_calf_joint" type="revolute">
+        <joint name="${prefix}${name}_calf_joint" type="revolute">
             <origin rpy="0 0 0" xyz="0 0 ${-thigh_length}"/>
-            <parent link="${name}_thigh"/>
-            <child link="${name}_calf"/>
+            <parent link="${prefix}${name}_thigh"/>
+            <child link="${prefix}${name}_calf"/>
             <axis xyz="0 1 0"/>
             <dynamics damping="${damping}" friction="${friction}"/>
             <limit effort="${calf_torque_max}" velocity="${calf_velocity_max}" lower="${calf_min*PI/180.0}" upper="${calf_max*PI/180.0}"/>
         </joint>
-        <link name="${name}_calf">
+        <link name="${prefix}${name}_calf">
             <visual>
                 <origin rpy="0 0 0" xyz="0 0 0"/>
@@ -130,10 +130,10 @@
             </inertial>
         </link>
-        <joint name="${name}_foot_fixed" type="fixed">
+        <joint name="${prefix}${name}_foot_fixed" type="fixed">
             <origin rpy="0 0 0" xyz="0 0 ${-(calf_length)}"/>
-            <parent link="${name}_calf"/>
-            <child link="${name}_foot"/>
+            <parent link="${prefix}${name}_calf"/>
+            <child link="${prefix}${name}_foot"/>
         </joint>
-        <link name="${name}_foot">
+        <link name="${prefix}${name}_foot">
             <visual>
                 <origin rpy="0 0 0" xyz="0 0 0"/>

File: arena_robots/robots/go1/urdf/go1.urdf.xacro (robot description, xacro)
@@ -10,5 +10,5 @@
   <xacro:include filename="$(find arena_robots)/robots/go1/urdf/include/materials.xacro" />
   <xacro:include filename="$(find arena_robots)/robots/go1/urdf/include/leg.xacro" />
-  <link name="base">
+  <link name="$(arg prefix)base">
     <visual>
       <origin rpy="0 0 0" xyz="0 0 0"/>
@@ -18,10 +18,10 @@
     </visual>
   </link>
-  <joint name="floating_base" type="fixed">
+  <joint name="$(arg prefix)floating_base" type="fixed">
     <origin rpy="0 0 0" xyz="0 0 0"/>
-    <parent link="base"/>
-    <child link="trunk"/>
+    <parent link="$(arg prefix)base"/>
+    <child link="$(arg prefix)trunk"/>
   </joint>
-  <link name="trunk">
+  <link name="$(arg prefix)trunk">
     <visual>
       <origin rpy="0 0 0" xyz="0 0 0"/>
@@ -46,10 +46,10 @@
     </inertial>
   </link>
-  <joint name="imu_joint" type="fixed">
-    <parent link="trunk"/>
-    <child link="imu_link"/>
+  <joint name="$(arg prefix)imu_joint" type="fixed">
+    <parent link="$(arg prefix)trunk"/>
+    <child link="$(arg prefix)imu_link"/>
     <origin rpy="0 0 0" xyz="-0.01592 -0.06659 -0.00617"/>
   </joint>
-  <link name="imu_link">
+  <link name="$(arg prefix)imu_link">
     <inertial>
       <mass value="0.001"/>
@@ -58,18 +58,18 @@
     </inertial>
   </link>
-  <xacro:leg name="FR" mirror="-1" mirror_dae="False" front_hind="1" front_hind_dae="True">
+  <xacro:leg name="FR" prefix="$(arg prefix)" mirror="-1" mirror_dae="False" front_hind="1" front_hind_dae="True">
     <origin rpy="0 0 0" xyz="${leg_offset_x} ${-leg_offset_y} 0"/>
   </xacro:leg>
-  <xacro:leg name="FL" mirror="1" mirror_dae="True" front_hind="1" front_hind_dae="True">
+  <xacro:leg name="FL" prefix="$(arg prefix)" mirror="1" mirror_dae="True" front_hind="1" front_hind_dae="True">
     <origin rpy="0 0 0" xyz="${leg_offset_x} ${leg_offset_y} 0"/>
   </xacro:leg>
-  <xacro:leg name="RR" mirror="-1" mirror_dae="False" front_hind="-1" front_hind_dae="False">
+  <xacro:leg name="RR" prefix="$(arg prefix)" mirror="-1" mirror_dae="False" front_hind="-1" front_hind_dae="False">
     <origin rpy="0 0 0" xyz="${-leg_offset_x} ${-leg_offset_y} 0"/>
   </xacro:leg>
-  <xacro:leg name="RL" mirror="1" mirror_dae="True" front_hind="-1" front_hind_dae="False">
+  <xacro:leg name="RL" prefix="$(arg prefix)" mirror="1" mirror_dae="True" front_hind="-1" front_hind_dae="False">
     <origin rpy="0 0 0" xyz="${-leg_offset_x} ${leg_offset_y} 0"/>
   </xacro:leg>
   <xacro:include filename="$(find arena_robots)/robots/go1/urdf/base_hw/go1.ros2_control.urdf" />
-  <xacro:go1_base_hw_controller/>
+  <xacro:go1_base_hw_controller prefix="$(arg prefix)"/>
   <gazebo>
     <plugin filename="libgz_ros2_control-system.so" name="gz_ros2_control::GazeboSimROS2ControlPlugin">
@@ -92,6 +92,6 @@
   </gazebo>
   <!-- Foot traction: legged stance needs high friction at the contact spheres. -->
-  <xacro:macro name="foot_friction" params="leg">
-    <gazebo reference="${leg}_foot">
+  <xacro:macro name="foot_friction" params="leg prefix">
+    <gazebo reference="${prefix}${leg}_foot">
       <mu1>0.8</mu1>
       <mu2>0.8</mu2>
@@ -100,7 +100,7 @@
     </gazebo>
   </xacro:macro>
-  <xacro:foot_friction leg="FL"/>
-  <xacro:foot_friction leg="FR"/>
-  <xacro:foot_friction leg="RL"/>
-  <xacro:foot_friction leg="RR"/>
+  <xacro:foot_friction leg="FL" prefix="$(arg prefix)"/>
+  <xacro:foot_friction leg="FR" prefix="$(arg prefix)"/>
+  <xacro:foot_friction leg="RL" prefix="$(arg prefix)"/>
+  <xacro:foot_friction leg="RR" prefix="$(arg prefix)"/>
 </robot>

File: arena_robots/robots/go1/urdf/include/depthcamera.xacro (robot description, xacro)
@@ -5,11 +5,11 @@
 <robot xmlns:xacro="http://www.ros.org/wiki/xacro">
   <xacro:include filename="$(find arena_robots)/urdf/gz_rgbd_camera.xacro"/>
-  <xacro:macro name="go1_depth_camera" params="camID name *origin">
-    <joint name="camera_joint_${name}" type="fixed">
+  <xacro:macro name="go1_depth_camera" params="camID name prefix:='' *origin">
+    <joint name="${prefix}camera_joint_${name}" type="fixed">
       <xacro:insert_block name="origin"/>
-      <parent link="trunk"/>
-      <child link="camera_${name}"/>
+      <parent link="${prefix}trunk"/>
+      <child link="${prefix}camera_${name}"/>
     </joint>
-    <link name="camera_${name}">
+    <link name="${prefix}camera_${name}">
       <collision>
         <origin xyz="0 0 0" rpy="0 0 0"/>
@@ -31,11 +31,11 @@
       </inertial>
     </link>
-    <joint name="camera_optical_joint_${name}" type="fixed">
+    <joint name="${prefix}camera_optical_joint_${name}" type="fixed">
       <origin xyz="0 0 0" rpy="${-pi/2} 0 ${-pi/2}"/>
-      <parent link="camera_${name}"/>
-      <child link="camera_optical_${name}"/>
+      <parent link="${prefix}camera_${name}"/>
+      <child link="${prefix}camera_optical_${name}"/>
     </joint>
-    <link name="camera_optical_${name}"/>
-    <xacro:gz_rgbd_camera frame="camera_${name}" sensor_name="camera_${name}"
+    <link name="${prefix}camera_optical_${name}"/>
+    <xacro:gz_rgbd_camera frame="${prefix}camera_${name}" sensor_name="${prefix}camera_${name}"
                           fov="2.094" width="928" height="800" near="0.1" far="5.0"
                           update_rate="16" pose="0.04 0 0 0 0 0"/>

File: arena_robots/robots/go1/urdf/include/leg.xacro (robot description, xacro)
@@ -1,9 +1,9 @@
 <?xml version="1.0"?>
 <robot xmlns:xacro="http://www.ros.org/wiki/xacro">
-    <xacro:macro name="leg" params="name mirror mirror_dae front_hind front_hind_dae *origin">
-        <joint name="${name}_hip_joint" type="revolute">
+    <xacro:macro name="leg" params="name prefix mirror mirror_dae front_hind front_hind_dae *origin">
+        <joint name="${prefix}${name}_hip_joint" type="revolute">
             <xacro:insert_block name="origin"/>
-            <parent link="trunk"/>
-            <child link="${name}_hip"/>
+            <parent link="${prefix}trunk"/>
+            <child link="${prefix}${name}_hip"/>
             <axis xyz="1 0 0"/>
             <dynamics damping="${damping}" friction="${friction}"/>
@@ -15,5 +15,5 @@
             </xacro:if>
         </joint>
-        <link name="${name}_hip">
+        <link name="${prefix}${name}_hip">
             <visual>
                 <xacro:if value="${(mirror_dae == True) and (front_hind_dae == True)}">
@@ -49,11 +49,11 @@
             </inertial>
         </link>
-        <joint name="${name}_hip_fixed" type="fixed">
+        <joint name="${prefix}${name}_hip_fixed" type="fixed">
             <origin rpy="0 0 0" xyz="0 ${(hip_offset)*mirror} 0"/>
-            <parent link="${name}_hip"/>
-            <child link="${name}_thigh_shoulder"/>
+            <parent link="${prefix}${name}_hip"/>
+            <child link="${prefix}${name}_thigh_shoulder"/>
         </joint>
         <!-- this link is only for collision -->
-        <link name="${name}_thigh_shoulder">
+        <link name="${prefix}${name}_thigh_shoulder">
             <collision>
                 <origin rpy="${PI/2.0} 0 0" xyz="0 0 0"/>
@@ -63,13 +63,13 @@
             </collision>
         </link>
-        <joint name="${name}_thigh_joint" type="revolute">
+        <joint name="${prefix}${name}_thigh_joint" type="revolute">
             <origin rpy="0 0 0" xyz="0 ${thigh_offset*mirror} 0"/>
-            <parent link="${name}_hip"/>
-            <child link="${name}_thigh"/>
+            <parent link="${prefix}${name}_hip"/>
+            <child link="${prefix}${name}_thigh"/>
             <axis xyz="0 1 0"/>
             <dynamics damping="${damping}" friction="${friction}"/>
             <limit effort="${thigh_torque_max}" velocity="${thigh_velocity_max}" lower="${thigh_min*PI/180.0}" upper="${thigh_max*PI/180.0}"/>
         </joint>
-        <link name="${name}_thigh">
+        <link name="${prefix}${name}_thigh">
             <visual>
                 <origin rpy="0 0 0" xyz="0 0 0"/>
@@ -99,13 +99,13 @@
             </inertial>
         </link>
-        <joint name="${name}_calf_joint" type="revolute">
+        <joint name="${prefix}${name}_calf_joint" type="revolute">
             <origin rpy="0 0 0" xyz="0 0 ${-thigh_length}"/>
-            <parent link="${name}_thigh"/>
-            <child link="${name}_calf"/>
+            <parent link="${prefix}${name}_thigh"/>
+            <child link="${prefix}${name}_calf"/>
             <axis xyz="0 1 0"/>
             <dynamics damping="${damping}" friction="${friction}"/>
             <limit effort="${calf_torque_max}" velocity="${calf_velocity_max}" lower="${calf_min*PI/180.0}" upper="${calf_max*PI/180.0}"/>
         </joint>
-        <link name="${name}_calf">
+        <link name="${prefix}${name}_calf">
             <visual>
                 <origin rpy="0 0 0" xyz="0 0 0"/>
@@ -130,10 +130,10 @@
             </inertial>
         </link>
-        <joint name="${name}_foot_fixed" type="fixed">
+        <joint name="${prefix}${name}_foot_fixed" type="fixed">
             <origin rpy="0 0 0" xyz="0 0 ${-(calf_length)}"/>
-            <parent link="${name}_calf"/>
-            <child link="${name}_foot"/>
+            <parent link="${prefix}${name}_calf"/>
+            <child link="${prefix}${name}_foot"/>
         </joint>
-        <link name="${name}_foot">
+        <link name="${prefix}${name}_foot">
             <visual>
                 <origin rpy="0 0 0" xyz="0 0 0"/>
