Commit message: migrate jackal, rbsummit, turtlebot, husky, dingo, WLP311D, WLP311E

File: arena_robots/robots/WLP311D/urdf/WLP311D.urdf.xacro (robot description, xacro)
@@ -6,6 +6,7 @@
 <robot name="WLP311D" xmlns:xacro="http://wiki.ros.org/xacro">
     <xacro:arg name="namespace" default=""/>
-    <xacro:include filename="$(find arena_robots)/config/urdf/sensors/default.xacro"/>
-    <xacro:arena_default_nav_sensors parent_link="base"/>
+    <xacro:arg name="prefix" default=""/>
+    <xacro:arg name="gazebo_classic" default="false"/>
+    <xacro:arg name="gazebo_ignition" default="true"/>
     <material name="black">
         <color rgba="0.0 0.0 0.0 1.0" />

File: arena_robots/robots/WLP311E/urdf/WLP311E.urdf.xacro (robot description, xacro)
@@ -6,6 +6,7 @@
 <robot name="WLP311E" xmlns:xacro="http://wiki.ros.org/xacro">
     <xacro:arg name="namespace" default=""/>
-    <xacro:include filename="$(find arena_robots)/config/urdf/sensors/default.xacro"/>
-    <xacro:arena_default_nav_sensors parent_link="base"/>
+    <xacro:arg name="prefix" default=""/>
+    <xacro:arg name="gazebo_classic" default="false"/>
+    <xacro:arg name="gazebo_ignition" default="true"/>
     <material name="black">
         <color rgba="0.0 0.0 0.0 1.0" />

File: arena_robots/robots/dingo/urdf/dingo-d.urdf.xacro (robot description, xacro)
@@ -218,9 +218,8 @@
     <child link="front_bumper_mount" />
   </joint>
-  <!-- gz-sim sensors; imu_link is already used for the kinematic frame -->
-  <xacro:arg name="sim_path" default=""/>
-  <xacro:include filename="$(find arena_robots)/config/urdf/sensors/default.xacro"/>
-  <xacro:arena_default_lidar parent_link="base_link"/>
-  <xacro:arena_default_imu parent_link="base_link" frame="imu_sensor_link"/>
+  <xacro:arg name="namespace" default=""/>
+  <xacro:arg name="prefix" default=""/>
+  <xacro:arg name="gazebo_classic" default="false"/>
+  <xacro:arg name="gazebo_ignition" default="true"/>
   <!-- PACS -->
   <xacro:include filename="$(find arena_robots)/robots/dingo/urdf/pacs.urdf.xacro"/>

File: arena_robots/robots/husky/urdf/husky.urdf.xacro (robot description, xacro)
@@ -325,9 +325,8 @@
     <xacro:outdoornav_sensors outdoornav_configuration="$(arg outdoornav_configuration)" />
   </xacro:if>
-  <!-- gz-sim sensors; imu_link is already used for the kinematic frame -->
-  <xacro:arg name="sim_path" default=""/>
-  <xacro:include filename="$(find arena_robots)/config/urdf/sensors/default.xacro"/>
-  <xacro:arena_default_lidar parent_link="base_link"/>
-  <xacro:arena_default_imu parent_link="base_link" frame="imu_sensor_link"/>
+  <xacro:arg name="namespace" default=""/>
+  <xacro:arg name="prefix" default=""/>
+  <xacro:arg name="gazebo_classic" default="false"/>
+  <xacro:arg name="gazebo_ignition" default="true"/>
   <xacro:husky_base_hw_controller/>
   <gazebo>

File: arena_robots/robots/jackal/urdf/jackal.urdf.xacro (robot description, xacro)
@@ -5,4 +5,6 @@
   <xacro:arg name="namespace" default="" />
   <xacro:arg name="gazebo_controllers" default="" />
+  <xacro:arg name="gazebo_classic" default="false" />
+  <xacro:arg name="gazebo_ignition" default="true" />
   <xacro:property name="PI" value="3.1415926535897931" />
   <xacro:property name="wheelbase" value="0.262" />
@@ -15,5 +17,4 @@
   <xacro:property name="chassis_width" value="0.310" />
   <xacro:property name="chassis_height" value="0.184" />
-  <xacro:property name="dummy_inertia" value="1e-09"/>
   <xacro:property name="mount_spacing" value="0.120" />
   <material name="dark_grey"><color rgba="0.2 0.2 0.2 1.0" /></material>
@@ -177,49 +178,7 @@
     <child link="rear_fender_link" />
   </joint>
-  <!-- TODO: Make this internal_imu_link or something, and use a mixed-in xacro
-       to supply the joint between it and imu_link. This is important so that imu_link
-       always points to the "active" IMU. When an upgrade IMU is connected, the
-       internal_imu_link should remain, but imu_link should point to the upgrade one. -->
-  <link name="imu_link">
-    <inertial>
-      <mass value="0.001"/>
-      <origin xyz="0 0 0" rpy="0 0 0"/>
-      <inertia ixx="${dummy_inertia}" ixy="0.0" ixz="0.0" iyy="${dummy_inertia}" iyz="0.0" izz="${dummy_inertia}"/>
-    </inertial>
-  </link>
-  <joint name="imu_joint" type="fixed">
-    <parent link="chassis_link" />
-    <child link="imu_link" />
-  </joint>
   <frame name="lidar_frame" attached_to="chassis_link">
     <pose>0.0 0.0 ${chassis_height/2 + 0.05} 0 0 0</pose>
   </frame>
-  <link name="lidar_link">
-      <inertial>
-          <origin xyz="0 0 0" rpy="0 0 0"/>
-          <mass value="0.1"/>
-          <inertia ixx="1e-5" ixy="0" ixz="0" iyy="1e-5" iyz="0" izz="1e-5"/>
-      </inertial>
-      <visual>
-          <origin xyz="0 0 0" rpy="0 0 0"/>
-          <geometry>
-              <cylinder radius="0.05" length="0.1"/>
-          </geometry>
-          <material name="black"/>
-      </visual>
-      <collision>
-          <origin xyz="0 0 0" rpy="0 0 0"/>
-          <geometry>
-              <cylinder radius="0.05" length="0.1"/>
-          </geometry>
-      </collision>
-  </link>
-  <!-- Fixed joint to attach the LiDAR to the chassis -->
-  <joint name="lidar_joint" type="fixed">
-      <parent link="chassis_link"/>
-      <child link="lidar_link"/>
-      <origin xyz="0.0 0.0 ${chassis_height/2 + 0.05}" rpy="0 0 0"/>
-  </joint>
-  <!-- TODO: Same note as applies to imu_link -->
   <link name="navsat_link">
     <visual>

File: arena_robots/robots/mpo700/urdf/mpo700.urdf.xacro (robot description, xacro)
@@ -13,6 +13,4 @@
   <xacro:include filename="$(find arena_robots)/robots/rbvogui/urdf/utils/inertia.urdf.xacro"/>
   <xacro:mpo_700_body/>
-  <!-- SENSORS: migrated to the component catalog (assembly.yaml, Stage M); attached
-       by the per-robot wrapper xacro (catalog.render_wrapper_xacro), not here. -->
   <xacro:mpo700_base_hw_controller/>
 </robot>

File: arena_robots/robots/rbrobout/urdf/rbrobout.urdf.xacro (robot description, xacro)
@@ -16,6 +16,4 @@
   <xacro:arg name="gazebo_controllers" default=""/>
   <xacro:rbrobout prefix="$(arg prefix)" gazebo_ignition="$(arg gazebo_ignition)"/>
-  <!-- SENSORS: migrated to the component catalog (assembly.yaml, Stage M); attached
-       by the per-robot wrapper xacro (catalog.render_wrapper_xacro), not here. -->
   <!-- ros2_control hardware block (always active; gz plugin loaded via rbrobout.gazebo) -->
   <xacro:rbrobout_base_hw_controller/>

File: arena_robots/robots/rbsummit/urdf/rbsummit.urdf.xacro (robot description, xacro)
@@ -20,13 +20,4 @@
 	<xacro:arg name="gazebo_classic" default="false"/>
 	<xacro:arg name="gazebo_ignition" default="true"/>
-	<xacro:property name="imu_offset_x" value="0.0385"/>
-	<xacro:property name="imu_offset_y" value="0.132"/>
-	<xacro:property name="imu_offset_z" value="0.158"/>
-	<xacro:property name="top_laser_offset_x" value="-0.01924"/>
-	<xacro:property name="top_laser_offset_y" value="0.0"/>
-	<xacro:property name="top_laser_offset_z" value="0.27642"/>
-	<xacro:property name="front_rgbd_camera_offset_x" value="0.324"/>
-	<xacro:property name="front_rgbd_camera_offset_y" value="0.012"/>
-	<xacro:property name="front_rgbd_camera_offset_z" value="0.172"/>
 	<xacro:property name="gps_offset_x" value="-0.22528"/>
 	<xacro:property name="gps_offset_y" value="0.095"/>
@@ -37,37 +28,4 @@
 	<!-- Here we create the robot using the xacro:macro imported at the beggining of this file -->
 	<xacro:rbsummit prefix="$(arg prefix)" hq="${hq}"/>
-	<!-- Custom Sensors -->
-	<!-- IMU -->
-    <xacro:sensor_vectornav
-        frame_prefix="$(arg prefix)vectornav_"
-        parent="$(arg prefix)base_link"
-        node_namespace="$(arg namespace)"
-        gazebo_classic="$(arg gazebo_classic)"
-        gazebo_ignition="$(arg gazebo_ignition)">
-        <origin xyz="${imu_offset_x} ${imu_offset_y} ${imu_offset_z}" rpy="0 0 0"/>
-    </xacro:sensor_vectornav>
-	<!-- 3D LIDAR -->
-	<xacro:sensor_robosense_helios_16p
-		frame_prefix="$(arg prefix)top_3d_laser_"
-		parent="$(arg prefix)base_link"
-        node_namespace="$(arg namespace)"
-        node_name="top_lidar"
-        gazebo_classic="$(arg gazebo_classic)"
-        gazebo_ignition="$(arg gazebo_ignition)">
-		<origin
-			xyz="${top_laser_offset_x} ${top_laser_offset_y} ${top_laser_offset_z}"
-			rpy="0 0 0"
-		/>
-	</xacro:sensor_robosense_helios_16p>
-	<!-- CAMERA -->
-    <xacro:sensor_intel_realsense_d435
-        frame_prefix="$(arg prefix)front_rgbd_camera_"
-        parent="$(arg prefix)base_link"
-        node_namespace="$(arg namespace)"
-        node_name="front_camera"
-        gazebo_classic="$(arg gazebo_classic)"
-        gazebo_ignition="$(arg gazebo_ignition)">
-        <origin xyz="${front_rgbd_camera_offset_x} ${front_rgbd_camera_offset_y} ${front_rgbd_camera_offset_z}" rpy="0 0 0"/>
-    </xacro:sensor_intel_realsense_d435>
 	<!-- GPS -->
 	<xacro:sensor_ublox_with_mast

File: arena_robots/robots/rbtheron/urdf/rbtheron.urdf.xacro (robot description, xacro)
@@ -27,6 +27,4 @@
 	<!-- Here we create the robot using the xacro:macro imported at the beggining of this file -->
 	<xacro:rbtheron prefix="$(arg prefix)" hq="${hq}"/>
-	<!-- SENSORS: migrated to the component catalog (assembly.yaml, Stage M); attached
-	     by the per-robot wrapper xacro (catalog.render_wrapper_xacro), not here. -->
 	<!-- Controllers -->
 	<xacro:if value="$(arg gazebo_classic)">

File: arena_robots/robots/rbvogui/urdf/rbvogui.urdf.xacro (robot description, xacro)
@@ -23,6 +23,4 @@
 	<xacro:arg name="generate_ros2_control_tag" default="true"/>
     <xacro:rbvogui prefix="$(arg prefix)" hq="${hq}"/>
-    <!-- SENSORS: migrated to the component catalog (assembly.yaml, Stage M); attached
-         by the per-robot wrapper xacro (catalog.render_wrapper_xacro), not here. -->
     <!-- ros2_control block (gz_ros2_control/GazeboSimSystem) and PosePublisher loaded via rbvogui.gazebo -->
     <xacro:if value="$(arg generate_ros2_control_tag)">

File: arena_robots/robots/ridgeback/urdf/ridgeback.urdf.xacro (robot description, xacro)
@@ -288,6 +288,4 @@
   <xacro:include filename="$(find arena_robots)/robots/ridgeback/urdf/base_hw/ridgeback.ros2_control.urdf"/>
   <xacro:include filename="$(find arena_robots)/robots/ridgeback/urdf/ridgeback.gazebo" />
-  <!-- SENSORS: migrated to the component catalog (assembly.yaml, Stage M); attached
-       by the per-robot wrapper xacro (catalog.render_wrapper_xacro), not here. -->
   <xacro:arg name="namespace" default=""/>
   <xacro:arg name="prefix" default=""/>

File: arena_robots/robots/rskomnidirectional/urdf/rskomnidirectional.urdf.xacro (robot description, xacro)
@@ -8,6 +8,4 @@
   <xacro:arg name="gazebo_classic" default="false"/>
   <xacro:arg name="gazebo_ignition" default="true"/>
-  <!-- SENSORS: migrated to the component catalog (assembly.yaml, Stage M); attached
-       by the per-robot wrapper xacro (catalog.render_wrapper_xacro), not here. -->
   <xacro:include filename="$(find arena_robots)/robots/rskomnidirectional/urdf/base_hw/rskomnidirectional.ros2_control.urdf"/>
   <xacro:rskomnidirectional_base_hw_controller/>

File: arena_robots/robots/turtlebot/urdf/turtlebot.urdf.xacro (robot description, xacro)
@@ -2,12 +2,13 @@
 <robot name="turtlebot" xmlns:xacro="http://ros.org/wiki/xacro">
   <xacro:arg name="namespace" default=""/>
+  <xacro:arg name="prefix" default=""/>
   <xacro:arg name="gazebo_controllers" default=""/>
   <xacro:arg name="sim_path" default=""/>
+  <xacro:arg name="gazebo_classic" default="false"/>
+  <xacro:arg name="gazebo_ignition" default="true"/>
   <!-- Base create3 model -->
   <xacro:include filename="$(find irobot_create_description)/urdf/create3.urdf.xacro">
     <xacro:arg name="gazebo" value="ignition"/>
   </xacro:include>
-  <xacro:include filename="$(find arena_robots)/robots/turtlebot/urdf/sensors/rplidar.urdf.xacro" />
-  <xacro:include filename="$(find arena_robots)/robots/turtlebot/urdf/sensors/oakd.urdf.xacro" />
   <xacro:include filename="$(find arena_robots)/robots/turtlebot/urdf/sensors/camera_bracket.urdf.xacro" />
   <xacro:include filename="$(find arena_robots)/robots/turtlebot/urdf/tower_standoff.urdf.xacro" />
@@ -100,13 +101,7 @@
   </xacro:tower_sensor_plate>
   <!-- Sensors -->
-  <xacro:rplidar name="rplidar" parent_link="shell_link" gazebo="true">
-    <origin xyz="${rplidar_x_offset} ${rplidar_y_offset} ${rplidar_z_offset}" rpy="0 0 ${pi/2}"/>
-  </xacro:rplidar>
   <xacro:camera_bracket name="oakd_camera_bracket">
     <origin xyz="${camera_mount_x_offset} ${camera_mount_y_offset} ${camera_mount_z_offset}"/>
   </xacro:camera_bracket>
-  <xacro:oakd model="pro" parent_link="oakd_camera_bracket">
-    <origin xyz="${oakd_pro_x_offset} ${oakd_pro_y_offset} ${oakd_pro_z_offset}"/>
-  </xacro:oakd>
   <xacro:turtlebot_base_hw_controller/>
   <!-- Wheel Friction and Dynamics -->

Commit message: fix WLP311D

File: arena_robots/robots/WLP311D/urdf/WLP311D.urdf.xacro (robot description, xacro)
@@ -7,6 +7,17 @@
     <xacro:arg name="namespace" default=""/>
     <xacro:arg name="prefix" default=""/>
+    <xacro:arg name="gazebo_controllers" default=""/>
     <xacro:arg name="gazebo_classic" default="false"/>
     <xacro:arg name="gazebo_ignition" default="true"/>
+    <xacro:include filename="$(find arena_robots)/robots/WLP311D/urdf/base_hw/WLP311D.ros2_control.urdf"/>
+    <xacro:wlp311d_base_hw_controller/>
+    <gazebo>
+        <plugin filename="libgz_ros2_control-system.so" name="gz_ros2_control::GazeboSimROS2ControlPlugin">
+            <parameters>$(arg gazebo_controllers)</parameters>
+            <ros>
+                <namespace>$(arg namespace)</namespace>
+            </ros>
+        </plugin>
+    </gazebo>
     <material name="black">
         <color rgba="0.0 0.0 0.0 1.0" />
@@ -67,6 +78,7 @@
     </gazebo>
     <gazebo reference="LF_wheel">
-        <mu1>0.6</mu1>
-        <mu2>0.6</mu2>
+        <mu1>0.35</mu1>
+        <mu2>1.0</mu2>
+        <fdir1>0 0 1</fdir1>
         <self_collide>1</self_collide>
         <material>Gazebo/DarkGrey</material>
@@ -102,6 +114,7 @@
     </gazebo>
     <gazebo reference="RF_wheel">
-        <mu1>0.6</mu1>
-        <mu2>0.6</mu2>
+        <mu1>0.35</mu1>
+        <mu2>1.0</mu2>
+        <fdir1>0 0 1</fdir1>
         <self_collide>1</self_collide>
         <material>Gazebo/DarkGrey</material>
@@ -137,6 +150,7 @@
     </gazebo>
     <gazebo reference="LH_wheel">
-        <mu1>0.6</mu1>
-        <mu2>0.6</mu2>
+        <mu1>0.35</mu1>
+        <mu2>1.0</mu2>
+        <fdir1>0 0 1</fdir1>
         <self_collide>1</self_collide>
         <material>Gazebo/DarkGrey</material>
@@ -172,6 +186,7 @@
     </gazebo>
     <gazebo reference="RH_wheel">
-        <mu1>0.6</mu1>
-        <mu2>0.6</mu2>
+        <mu1>0.35</mu1>
+        <mu2>1.0</mu2>
+        <fdir1>0 0 1</fdir1>
         <self_collide>1</self_collide>
         <material>Gazebo/DarkGrey</material>
@@ -325,10 +340,10 @@
         </inertial>
     </link>
-    <joint name="LF_WHL" type="revolute">
+    <joint name="LF_WHL" type="continuous">
         <origin rpy="0 0 0" xyz="0.21449 0.03434 -0.17998" />
         <parent link="LF_calf" />
         <child link="LF_wheel" />
         <axis xyz="0 1 0" />
-        <limit effort="40" lower="-1000" upper="1000" velocity="20" />
+        <limit effort="40" velocity="20" />
         <dynamics friction="1" />
     </joint>
@@ -502,10 +517,10 @@
         </inertial>
     </link>
-    <joint name="RF_WHL" type="revolute">
+    <joint name="RF_WHL" type="continuous">
         <origin rpy="0 0 0" xyz="0.21449 -0.03434 -0.17998" />
         <parent link="RF_calf" />
         <child link="RF_wheel" />
         <axis xyz="0 1 0" />
-        <limit effort="40" lower="-1000" upper="1000" velocity="20" />
+        <limit effort="40" velocity="20" />
         <dynamics friction="1" />
     </joint>
@@ -679,10 +694,10 @@
         </inertial>
     </link>
-    <joint name="LH_WHL" type="revolute">
+    <joint name="LH_WHL" type="continuous">
         <origin rpy="0 0 0" xyz="0.21449 0.03434 -0.17998" />
         <parent link="LH_calf" />
         <child link="LH_wheel" />
         <axis xyz="0 1 0" />
-        <limit effort="40" lower="-1000" upper="1000" velocity="20" />
+        <limit effort="40" velocity="20" />
         <dynamics friction="1" />
     </joint>
@@ -856,10 +871,10 @@
         </inertial>
     </link>
-    <joint name="RH_WHL" type="revolute">
+    <joint name="RH_WHL" type="continuous">
         <origin rpy="0 0 0" xyz="0.21449 -0.03434 -0.17998" />
         <parent link="RH_calf" />
         <child link="RH_wheel" />
         <axis xyz="0 1 0" />
-        <limit effort="40" lower="-1000" upper="1000" velocity="20" />
+        <limit effort="40" velocity="20" />
         <dynamics friction="1" />
     </joint>

File: arena_robots/tests/golden/WLP311D_default.urdf (robot description, URDF)
Before this commit: robot WLP311D, 24 links, 23 joints
Joints:
- joint LF_WHL: limit lower=-1000 upper=1000 effort=40 velocity=20 -> effort=40 velocity=20; type revolute -> continuous
- joint LH_WHL: limit lower=-1000 upper=1000 effort=40 velocity=20 -> effort=40 velocity=20; type revolute -> continuous
- joint RF_WHL: limit lower=-1000 upper=1000 effort=40 velocity=20 -> effort=40 velocity=20; type revolute -> continuous
- joint RH_WHL: limit lower=-1000 upper=1000 effort=40 velocity=20 -> effort=40 velocity=20; type revolute -> continuous
- joint imu_link_joint: origin xyz=0 0 0 rpy=0 0 0 -> xyz=0.0 0.0 0.0 rpy=0.0 0.0 0.0
- joint lidar_joint: origin xyz=0 0 0.3 rpy=0 0 0 -> xyz=0.0 0.0 0.3 rpy=0.0 0.0 0.0
