Commit message: fix WLP311E

File: arena_robots/robots/WLP311E/urdf/WLP311E.urdf.xacro (robot description, xacro)
@@ -7,6 +7,17 @@
     <xacro:arg name="namespace" default=""/>
     <xacro:arg name="prefix" default=""/>
+    <xacro:arg name="gazebo_controllers" default=""/>
     <xacro:arg name="gazebo_classic" default="false"/>
     <xacro:arg name="gazebo_ignition" default="true"/>
+    <xacro:include filename="$(find arena_robots)/robots/WLP311E/urdf/base_hw/WLP311E.ros2_control.urdf"/>
+    <xacro:wlp311e_base_hw_controller/>
+    <gazebo>
+        <plugin filename="libgz_ros2_control-system.so" name="gz_ros2_control::GazeboSimROS2ControlPlugin">
+            <parameters>$(arg gazebo_controllers)</parameters>
+            <ros>
+                <namespace>$(arg namespace)</namespace>
+            </ros>
+        </plugin>
+    </gazebo>
     <material name="black">
         <color rgba="0.0 0.0 0.0 1.0" />
@@ -67,6 +78,7 @@
     </gazebo>
     <gazebo reference="LF_wheel">
-        <mu1>0.6</mu1>
-        <mu2>0.6</mu2>
+        <mu1>0.35</mu1>
+        <mu2>1.0</mu2>
+        <fdir1>0 0 1</fdir1>
         <self_collide>1</self_collide>
         <material>Gazebo/DarkGrey</material>
@@ -102,6 +114,7 @@
     </gazebo>
     <gazebo reference="RF_wheel">
-        <mu1>0.6</mu1>
-        <mu2>0.6</mu2>
+        <mu1>0.35</mu1>
+        <mu2>1.0</mu2>
+        <fdir1>0 0 1</fdir1>
         <self_collide>1</self_collide>
         <material>Gazebo/DarkGrey</material>
@@ -137,6 +150,7 @@
     </gazebo>
     <gazebo reference="LH_wheel">
-        <mu1>0.6</mu1>
-        <mu2>0.6</mu2>
+        <mu1>0.35</mu1>
+        <mu2>1.0</mu2>
+        <fdir1>0 0 1</fdir1>
         <self_collide>1</self_collide>
         <material>Gazebo/DarkGrey</material>
@@ -172,6 +186,7 @@
     </gazebo>
     <gazebo reference="RH_wheel">
-        <mu1>0.6</mu1>
-        <mu2>0.6</mu2>
+        <mu1>0.35</mu1>
+        <mu2>1.0</mu2>
+        <fdir1>0 0 1</fdir1>
         <self_collide>1</self_collide>
         <material>Gazebo/DarkGrey</material>
@@ -313,10 +328,10 @@
         </inertial>
     </link>
-    <joint name="LF_WHL" type="revolute">
+    <joint name="LF_WHL" type="continuous">
         <origin rpy="0 -0.3 0" xyz="0.21449 0.03459 -0.17998" />
         <parent link="LF_calf" />
         <child link="LF_wheel" />
         <axis xyz="0 1 0" />
-        <limit effort="40" lower="-1000" upper="1000" velocity="20" />
+        <limit effort="40" velocity="20" />
         <dynamics friction="1" />
     </joint>
@@ -473,10 +488,10 @@
         </inertial>
     </link>
-    <joint name="RF_WHL" type="revolute">
+    <joint name="RF_WHL" type="continuous">
         <origin rpy="0 -0.3 0" xyz="0.21449 -0.03459 -0.17998" />
         <parent link="RF_calf" />
         <child link="RF_wheel" />
         <axis xyz="0 1 0" />
-        <limit effort="40" lower="-1000" upper="1000" velocity="20" />
+        <limit effort="40" velocity="20" />
         <dynamics friction="1" />
     </joint>
@@ -633,10 +648,10 @@
         </inertial>
     </link>
-    <joint name="LH_WHL" type="revolute">
+    <joint name="LH_WHL" type="continuous">
         <origin rpy="0 -0.3 0" xyz="0.21449 0.03459 -0.17998" />
         <parent link="LH_calf" />
         <child link="LH_wheel" />
         <axis xyz="0 1 0" />
-        <limit effort="40" lower="-1000" upper="1000" velocity="20" />
+        <limit effort="40" velocity="20" />
         <dynamics friction="1" />
     </joint>
@@ -793,10 +808,10 @@
         </inertial>
     </link>
-    <joint name="RH_WHL" type="revolute">
+    <joint name="RH_WHL" type="continuous">
         <origin rpy="0 -0.3 0" xyz="0.21449 -0.03459 -0.17998" />
         <parent link="RH_calf" />
         <child link="RH_wheel" />
         <axis xyz="0 1 0" />
-        <limit effort="40" lower="-1000" upper="1000" velocity="20" />
+        <limit effort="40" velocity="20" />
         <dynamics friction="1" />
     </joint>

File: arena_robots/tests/golden/WLP311E_default.urdf (robot description, URDF)
Before this commit: robot WLP311E, 24 links, 23 joints
Joints:
- joint LF_WHL: limit lower=-1000 upper=1000 effort=40 velocity=20 -> effort=40 velocity=20; type revolute -> continuous
- joint LH_WHL: limit lower=-1000 upper=1000 effort=40 velocity=20 -> effort=40 velocity=20; type revolute -> continuous
- joint RF_WHL: limit lower=-1000 upper=1000 effort=40 velocity=20 -> effort=40 velocity=20; type revolute -> continuous
- joint RH_WHL: limit lower=-1000 upper=1000 effort=40 velocity=20 -> effort=40 velocity=20; type revolute -> continuous
- joint imu_link_joint: origin xyz=0 0 0 rpy=0 0 0 -> xyz=0.0 0.0 0.0 rpy=0.0 0.0 0.0
- joint lidar_joint: origin xyz=0 0 0.3 rpy=0 0 0 -> xyz=0.0 0.0 0.3 rpy=0.0 0.0 0.0
