Commit message: fix rskomnidirectional

File: arena_robots/robots/rskomnidirectional/urdf/rskomnidirectional.urdf.xacro (robot description, xacro)
@@ -263,4 +263,10 @@
       </material>
     </visual>
+    <collision>
+      <origin xyz="0 0 -0.01" rpy="0 0 0"/>
+      <geometry>
+        <sphere radius="0.0345"/>
+      </geometry>
+    </collision>
   </link>
   <!-- Link pin_bearing_oring -->
@@ -274,10 +280,4 @@
     <!-- Part pin -->
     <!-- Part bearing -->
-    <collision>
-      <origin xyz="-4.17181e-17 9.00576e-17 -7.11237e-17" rpy="3.14159 -6.31857e-17 8.96642e-17"/>
-      <geometry>
-        <cylinder length="0.004" radius="0.006"/>
-      </geometry>
-    </collision>
     <visual>
       <origin xyz="-4.16334e-17 9.02056e-17 0.002" rpy="3.14159 -6.31857e-17 8.96642e-17"/>
@@ -291,10 +291,8 @@
   </link>
   <!-- Joint from wheel_no_passives to pin_bearing_oring -->
-  <joint name="wheel1_passive_1" type="continuous">
+  <joint name="wheel1_passive_1" type="fixed">
     <origin xyz="-0.00880698 0.0271051 -0.01" rpy="0.314159 -1.5708 0"/>
     <parent link="wheel_no_passives"/>
     <child link="pin_bearing_oring"/>
-    <axis xyz="0 0 1"/>
-    <limit effort="10" velocity="10"/>
   </joint>
   <!-- Link pin_bearing_oring_2 -->
@@ -308,10 +306,4 @@
     <!-- Part pin_2 -->
     <!-- Part bearing_2 -->
-    <collision>
-      <origin xyz="-6.70839e-18 6.24373e-17 -1.50921e-16" rpy="-3.14159 5.43994e-18 -2.56223e-17"/>
-      <geometry>
-        <cylinder length="0.004" radius="0.006"/>
-      </geometry>
-    </collision>
     <visual>
       <origin xyz="-6.93889e-18 6.245e-17 0.002" rpy="-3.14159 5.43994e-18 -2.56223e-17"/>
@@ -325,10 +317,8 @@
   </link>
   <!-- Joint from wheel_no_passives to pin_bearing_oring_2 -->
-  <joint name="wheel1_passive_2" type="continuous">
+  <joint name="wheel1_passive_2" type="fixed">
     <origin xyz="-0.0167519 0.023057 -0.01" rpy="-1.5708 2.93259e-16 -0.942478"/>
     <parent link="wheel_no_passives"/>
     <child link="pin_bearing_oring_2"/>
-    <axis xyz="0 0 1"/>
-    <limit effort="10" velocity="10"/>
   </joint>
   <!-- Link pin_bearing_oring_3 -->
@@ -342,10 +332,4 @@
     <!-- Part pin_3 -->
     <!-- Part bearing_3 -->
-    <collision>
-      <origin xyz="7.66345e-17 1.0425e-16 9.93129e-17" rpy="-3.91086e-16 4.44161e-16 -2.6898e-17"/>
-      <geometry>
-        <cylinder length="0.004" radius="0.006"/>
-      </geometry>
-    </collision>
     <visual>
       <origin xyz="7.63278e-17 1.04083e-16 -0.002" rpy="-3.91086e-16 4.44161e-16 -2.6898e-17"/>
@@ -359,10 +343,8 @@
   </link>
   <!-- Joint from wheel_no_passives to pin_bearing_oring_3 -->
-  <joint name="wheel1_passive_3" type="continuous">
+  <joint name="wheel1_passive_3" type="fixed">
     <origin xyz="-0.023057 0.0167519 -0.01" rpy="1.5708 -3.90162e-17 -0.628319"/>
     <parent link="wheel_no_passives"/>
     <child link="pin_bearing_oring_3"/>
-    <axis xyz="0 0 1"/>
-    <limit effort="10" velocity="10"/>
   </joint>
   <!-- Link pin_bearing_oring_4 -->
@@ -376,10 +358,4 @@
     <!-- Part pin_4 -->
     <!-- Part bearing_4 -->
-    <collision>
-      <origin xyz="-2.77544e-17 -2.08082e-17 -1.50487e-16" rpy="-3.14159 -1.4488e-18 -1.82407e-16"/>
-      <geometry>
-        <cylinder length="0.004" radius="0.006"/>
-      </geometry>
-    </collision>
     <visual>
       <origin xyz="-2.77556e-17 -2.08167e-17 0.002" rpy="-3.14159 -1.4488e-18 -1.82407e-16"/>
@@ -393,10 +369,8 @@
   </link>
   <!-- Joint from wheel_no_passives to pin_bearing_oring_4 -->
-  <joint name="wheel1_passive_4" type="continuous">
+  <joint name="wheel1_passive_4" type="fixed">
     <origin xyz="-0.0271051 0.00880698 -0.01" rpy="1.5708 -3.91234e-14 -0.314159"/>
     <parent link="wheel_no_passives"/>
     <child link="pin_bearing_oring_4"/>
-    <axis xyz="0 0 1"/>
-    <limit effort="10" velocity="10"/>
   </joint>
   <!-- Link pin_bearing_oring_5 -->
@@ -410,10 +384,4 @@
     <!-- Part pin_5 -->
     <!-- Part bearing_5 -->
-    <collision>
-      <origin xyz="1.11093e-16 2.22029e-16 -8.1532e-17" rpy="3.14159 4.46202e-17 6.08837e-17"/>
-      <geometry>
-        <cylinder length="0.004" radius="0.006"/>
-      </geometry>
-    </collision>
     <visual>
       <origin xyz="1.11022e-16 2.22045e-16 0.002" rpy="3.14159 4.46202e-17 6.08837e-17"/>
@@ -427,10 +395,8 @@
   </link>
   <!-- Joint from wheel_no_passives to pin_bearing_oring_5 -->
-  <joint name="wheel1_passive_5" type="continuous">
+  <joint name="wheel1_passive_5" type="fixed">
     <origin xyz="-0.0285 0 -0.01" rpy="1.5708 -6.94415e-14 -3.05443e-16"/>
     <parent link="wheel_no_passives"/>
     <child link="pin_bearing_oring_5"/>
-    <axis xyz="0 0 1"/>
-    <limit effort="10" velocity="10"/>
   </joint>
   <!-- Link pin_bearing_oring_6 -->
@@ -444,10 +410,4 @@
     <!-- Part pin_6 -->
     <!-- Part bearing_6 -->
-    <collision>
-      <origin xyz="-4.29413e-17 1.37484e-17 8.89046e-17" rpy="-6.37412e-16 4.21278e-16 -1.83796e-16"/>
-      <geometry>
-        <cylinder length="0.004" radius="0.006"/>
-      </geometry>
-    </collision>
     <visual>
       <origin xyz="-4.25007e-17 1.38778e-17 -0.002" rpy="-6.37412e-16 4.21278e-16 -1.83796e-16"/>
@@ -461,10 +421,8 @@
   </link>
   <!-- Joint from wheel_no_passives to pin_bearing_oring_6 -->
-  <joint name="wheel1_passive_6" type="continuous">
+  <joint name="wheel1_passive_6" type="fixed">
     <origin xyz="-0.0271051 -0.00880698 -0.01" rpy="1.5708 -5.27049e-17 0.314159"/>
     <parent link="wheel_no_passives"/>
     <child link="pin_bearing_oring_6"/>
-    <axis xyz="0 0 1"/>
-    <limit effort="10" velocity="10"/>
   </joint>
   <!-- Link pin_bearing_oring_7 -->
@@ -478,10 +436,4 @@
     <!-- Part pin_7 -->
     <!-- Part bearing_7 -->
-    <collision>
-      <origin xyz="-1.90034e-17 -8.33718e-17 -9.84456e-17" rpy="-3.14159 -2.2357e-17 -4.47672e-17"/>
-      <geometry>
-        <cylinder length="0.004" radius="0.006"/>
-      </geometry>
-    </collision>
     <visual>
       <origin xyz="-1.91904e-17 -8.32667e-17 0.002" rpy="-3.14159 -2.2357e-17 -4.47672e-17"/>
@@ -495,10 +447,8 @@
   </link>
   <!-- Joint from wheel_no_passives to pin_bearing_oring_7 -->
-  <joint name="wheel1_passive_7" type="continuous">
+  <joint name="wheel1_passive_7" type="fixed">
     <origin xyz="-0.023057 -0.0167519 -0.01" rpy="1.5708 -1.36878e-14 0.628319"/>
     <parent link="wheel_no_passives"/>
     <child link="pin_bearing_oring_7"/>
-    <axis xyz="0 0 1"/>
-    <limit effort="10" velocity="10"/>
   </joint>
   <!-- Link pin_bearing_oring_8 -->
@@ -512,10 +462,4 @@
     <!-- Part pin_8 -->
     <!-- Part bearing_8 -->
-    <collision>
-      <origin xyz="2.55746e-18 -7.64263e-17 -8.50015e-17" rpy="-3.14159 5.25847e-17 4.29229e-17"/>
-      <geometry>
-        <cylinder length="0.004" radius="0.006"/>
-      </geometry>
-    </collision>
     <visual>
       <origin xyz="2.60209e-18 -7.63278e-17 0.002" rpy="-3.14159 5.25847e-17 4.29229e-17"/>
@@ -529,10 +473,8 @@
   </link>
   <!-- Joint from wheel_no_passives to pin_bearing_oring_8 -->
-  <joint name="wheel1_passive_8" type="continuous">
+  <joint name="wheel1_passive_8" type="fixed">
     <origin xyz="-0.0167519 -0.023057 -0.01" rpy="1.5708 -1.74069e-15 0.942478"/>
     <parent link="wheel_no_passives"/>
     <child link="pin_bearing_oring_8"/>
-    <axis xyz="0 0 1"/>
-    <limit effort="10" velocity="10"/>
   </joint>
   <!-- Link pin_bearing_oring_9 -->
@@ -546,10 +488,4 @@
     <!-- Part pin_9 -->
     <!-- Part bearing_9 -->
-    <collision>
-      <origin xyz="5.57191e-17 -9.01972e-17 -9.80119e-17" rpy="3.14159 -4.88362e-18 -2.71284e-18"/>
-      <geometry>
-        <cylinder length="0.004" radius="0.006"/>
-      </geometry>
-    </collision>
     <visual>
       <origin xyz="5.55112e-17 -9.02056e-17 0.002" rpy="3.14159 -4.88362e-18 -2.71284e-18"/>
@@ -563,10 +499,8 @@
   </link>
   <!-- Joint from wheel_no_passives to pin_bearing_oring_9 -->
-  <joint name="wheel1_passive_9" type="continuous">
+  <joint name="wheel1_passive_9" type="fixed">
     <origin xyz="-0.00880698 -0.0271051 -0.01" rpy="-0.314159 -1.5708 0"/>
     <parent link="wheel_no_passives"/>
     <child link="pin_bearing_oring_9"/>
-    <axis xyz="0 0 1"/>
-    <limit effort="10" velocity="10"/>
   </joint>
   <!-- Link pin_bearing_oring_10 -->
@@ -580,10 +514,4 @@
     <!-- Part pin_10 -->
     <!-- Part bearing_10 -->
-    <collision>
-      <origin xyz="2.39153e-17 6.9364e-17 4.51028e-17" rpy="-1.92469e-16 -6.43876e-16 3.58098e-16"/>
-      <geometry>
-        <cylinder length="0.004" radius="0.006"/>
-      </geometry>
-    </collision>
     <visual>
       <origin xyz="2.42861e-17 6.93889e-17 -0.002" rpy="-1.92469e-16 -6.43876e-16 3.58098e-16"/>
@@ -597,10 +525,8 @@
   </link>
   <!-- Joint from wheel_no_passives to pin_bearing_oring_10 -->
-  <joint name="wheel1_passive_10" type="continuous">
+  <joint name="wheel1_passive_10" type="fixed">
     <origin xyz="1.73472e-18 -0.0285 -0.01" rpy="1.5708 -3.8774e-18 1.5708"/>
     <parent link="wheel_no_passives"/>
     <child link="pin_bearing_oring_10"/>
-    <axis xyz="0 0 1"/>
-    <limit effort="10" velocity="10"/>
   </joint>
   <!-- Link pin_bearing_oring_11 -->
@@ -614,10 +540,4 @@
     <!-- Part pin_11 -->
     <!-- Part bearing_11 -->
-    <collision>
-      <origin xyz="3.46581e-17 1.52241e-17 -1.23165e-16" rpy="-3.14159 -1.51665e-17 -5.96425e-17"/>
-      <geometry>
-        <cylinder length="0.004" radius="0.006"/>
-      </geometry>
-    </collision>
     <visual>
       <origin xyz="3.46945e-17 1.51788e-17 0.002" rpy="-3.14159 -1.51665e-17 -5.96425e-17"/>
@@ -631,10 +551,8 @@
   </link>
   <!-- Joint from wheel_no_passives to pin_bearing_oring_11 -->
-  <joint name="wheel1_passive_11" type="continuous">
+  <joint name="wheel1_passive_11" type="fixed">
     <origin xyz="0.00880698 -0.0271051 -0.01" rpy="0.314159 -1.5708 0"/>
     <parent link="wheel_no_passives"/>
     <child link="pin_bearing_oring_11"/>
-    <axis xyz="0 0 1"/>
-    <limit effort="10" velocity="10"/>
   </joint>
   <!-- Link pin_bearing_oring_12 -->
@@ -648,10 +566,4 @@
     <!-- Part pin_12 -->
     <!-- Part bearing_12 -->
-    <collision>
-      <origin xyz="-9.01926e-17 2.43399e-17 -1.12757e-16" rpy="3.14159 -1.73147e-17 1.16857e-17"/>
-      <geometry>
-        <cylinder length="0.004" radius="0.006"/>
-      </geometry>
-    </collision>
     <visual>
       <origin xyz="-9.02056e-17 2.42861e-17 0.002" rpy="3.14159 -1.73147e-17 1.16857e-17"/>
@@ -665,10 +577,8 @@
   </link>
   <!-- Joint from wheel_no_passives to pin_bearing_oring_12 -->
-  <joint name="wheel1_passive_12" type="continuous">
+  <joint name="wheel1_passive_12" type="fixed">
     <origin xyz="0.0167519 -0.023057 -0.01" rpy="0.628319 -1.5708 0"/>
     <parent link="wheel_no_passives"/>
     <child link="pin_bearing_oring_12"/>
-    <axis xyz="0 0 1"/>
-    <limit effort="10" velocity="10"/>
   </joint>
   <!-- Link pin_bearing_oring_13 -->
@@ -682,10 +592,4 @@
     <!-- Part pin_13 -->
     <!-- Part bearing_13 -->
-    <collision>
-      <origin xyz="-2.42785e-17 -1.38927e-17 -1.08854e-16" rpy="-3.14159 5.34155e-17 -5.25375e-17"/>
-      <geometry>
-        <cylinder length="0.004" radius="0.006"/>
-      </geometry>
-    </collision>
     <visual>
       <origin xyz="-2.42861e-17 -1.38778e-17 0.002" rpy="-3.14159 5.34155e-17 -5.25375e-17"/>
@@ -699,10 +603,8 @@
   </link>
   <!-- Joint from wheel_no_passives to pin_bearing_oring_13 -->
-  <joint name="wheel1_passive_13" type="continuous">
+  <joint name="wheel1_passive_13" type="fixed">
     <origin xyz="0.023057 -0.0167519 -0.01" rpy="1.5708 7.03424e-15 -0.628319"/>
     <parent link="wheel_no_passives"/>
     <child link="pin_bearing_oring_13"/>
-    <axis xyz="0 0 1"/>
-    <limit effort="10" velocity="10"/>
   </joint>
   <!-- Link pin_bearing_oring_14 -->
@@ -716,10 +618,4 @@
     <!-- Part pin_14 -->
     <!-- Part bearing_14 -->
-    <collision>
-      <origin xyz="-1.66541e-16 6.93866e-17 -3.29597e-17" rpy="-3.14159 4.44238e-19 2.05083e-17"/>
-      <geometry>
-        <cylinder length="0.004" radius="0.006"/>
-      </geometry>
-    </collision>
     <visual>
       <origin xyz="-1.66533e-16 6.93889e-17 0.002" rpy="-3.14159 4.44238e-19 2.05083e-17"/>
@@ -733,10 +629,8 @@
   </link>
   <!-- Joint from wheel_no_passives to pin_bearing_oring_14 -->
-  <joint name="wheel1_passive_14" type="continuous">
+  <joint name="wheel1_passive_14" type="fixed">
     <origin xyz="0.0271051 -0.00880698 -0.01" rpy="1.5708 7.48324e-15 -0.314159"/>
     <parent link="wheel_no_passives"/>
     <child link="pin_bearing_oring_14"/>
-    <axis xyz="0 0 1"/>
-    <limit effort="10" velocity="10"/>
   </joint>
   <!-- Link pin_bearing_oring_15 -->
@@ -750,10 +644,4 @@
     <!-- Part pin_15 -->
     <!-- Part bearing_15 -->
-    <collision>
-      <origin xyz="6.24243e-17 -7.63656e-17 -8.84709e-17" rpy="-3.14159 -1.15197e-17 6.94712e-17"/>
-      <geometry>
-        <cylinder length="0.004" radius="0.006"/>
-      </geometry>
-    </collision>
     <visual>
       <origin xyz="6.245e-17 -7.63278e-17 0.002" rpy="-3.14159 -1.15197e-17 6.94712e-17"/>
@@ -767,10 +655,8 @@
   </link>
   <!-- Joint from wheel_no_passives to pin_bearing_oring_15 -->
-  <joint name="wheel1_passive_15" type="continuous">
+  <joint name="wheel1_passive_15" type="fixed">
     <origin xyz="0.0285 -1.38778e-17 -0.01" rpy="1.5708 -2.63408e-14 -4.02599e-16"/>
     <parent link="wheel_no_passives"/>
     <child link="pin_bearing_oring_15"/>
-    <axis xyz="0 0 1"/>
-    <limit effort="10" velocity="10"/>
   </joint>
   <!-- Link pin_bearing_oring_16 -->
@@ -784,10 +670,4 @@
     <!-- Part pin_16 -->
     <!-- Part bearing_16 -->
-    <collision>
-      <origin xyz="4.13227e-17 1.41804e-17 1.32706e-16" rpy="1.78942e-15 -4.1326e-15 1.23498e-15"/>
-      <geometry>
-        <cylinder length="0.004" radius="0.006"/>
-      </geometry>
-    </collision>
     <visual>
       <origin xyz="4.16334e-17 1.38778e-17 -0.002" rpy="1.78942e-15 -4.1326e-15 1.23498e-15"/>
@@ -801,10 +681,8 @@
   </link>
   <!-- Joint from wheel_no_passives to pin_bearing_oring_16 -->
-  <joint name="wheel1_passive_16" type="continuous">
+  <joint name="wheel1_passive_16" type="fixed">
     <origin xyz="0.0271051 0.00880698 -0.01" rpy="1.5708 4.63079e-18 -2.82743"/>
     <parent link="wheel_no_passives"/>
     <child link="pin_bearing_oring_16"/>
-    <axis xyz="0 0 1"/>
-    <limit effort="10" velocity="10"/>
   </joint>
   <!-- Link pin_bearing_oring_17 -->
@@ -818,10 +696,4 @@
     <!-- Part pin_17 -->
     <!-- Part bearing_17 -->
-    <collision>
-      <origin xyz="3.55204e-17 3.5383e-17 1.18395e-16" rpy="1.54652e-16 -4.84388e-16 -6.60848e-16"/>
-      <geometry>
-        <cylinder length="0.004" radius="0.006"/>
-      </geometry>
-    </collision>
     <visual>
       <origin xyz="3.46945e-17 3.46945e-17 -0.002" rpy="1.54652e-16 -4.84388e-16 -6.60848e-16"/>
@@ -835,10 +707,8 @@
   </link>
   <!-- Joint from wheel_no_passives to pin_bearing_oring_17 -->
-  <joint name="wheel1_passive_17" type="continuous">
+  <joint name="wheel1_passive_17" type="fixed">
     <origin xyz="0.023057 0.0167519 -0.01" rpy="1.5708 6.01992e-17 -2.51327"/>
     <parent link="wheel_no_passives"/>
     <child link="pin_bearing_oring_17"/>
-    <axis xyz="0 0 1"/>
-    <limit effort="10" velocity="10"/>
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