Commit message: fix rskomnidirectional

File: arena_robots/tests/golden/rskomnidirectional_default.urdf (robot description, URDF)
Before this commit: robot urdf, 116 links, 115 joints
Links:
- link pin_bearing_oring: geometry visual mesh filename=package://arena_robots/robots/rskomnidirectional/meshes/bea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
- link pin_bearing_oring_10: geometry visual mesh filename=package://arena_robots/robots/rskomnidirectional/meshes/bea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
- link pin_bearing_oring_11: geometry visual mesh filename=package://arena_robots/robots/rskomnidirectional/meshes/bea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
- link pin_bearing_oring_12: geometry visual mesh filename=package://arena_robots/robots/rskomnidirectional/meshes/bea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
- link pin_bearing_oring_13: geometry visual mesh filename=package://arena_robots/robots/rskomnidirectional/meshes/bea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
- link pin_bearing_oring_14: geometry visual mesh filename=package://arena_robots/robots/rskomnidirectional/meshes/bea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
- link pin_bearing_oring_15: geometry visual mesh filename=package://arena_robots/robots/rskomnidirectional/meshes/bea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
- link pin_bearing_oring_16: geometry visual mesh filename=package://arena_robots/robots/rskomnidirectional/meshes/bea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
- link pin_bearing_oring_17: geometry visual mesh filename=package://arena_robots/robots/rskomnidirectional/meshes/bea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
- link pin_bearing_oring_18: geometry visual mesh filename=package://arena_robots/robots/rskomnidirectional/meshes/bea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
- link pin_bearing_oring_19: geometry visual mesh filename=package://arena_robots/robots/rskomnidirectional/meshes/bea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
- link pin_bearing_oring_2: geometry visual mesh filename=package://arena_robots/robots/rskomnidirectional/meshes/bea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
- link pin_bearing_oring_20: geometry visual mesh filename=package://arena_robots/robots/rskomnidirectional/meshes/bea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
- link pin_bearing_oring_21: geometry visual mesh filename=package://arena_robots/robots/rskomnidirectional/meshes/bea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
- link pin_bearing_oring_22: geometry visual mesh filename=package://arena_robots/robots/rskomnidirectional/meshes/bea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
- link pin_bearing_oring_23: geometry visual mesh filename=package://arena_robots/robots/rskomnidirectional/meshes/bea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
- link pin_bearing_oring_24: geometry visual mesh filename=package://arena_robots/robots/rskomnidirectional/meshes/bea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
- link pin_bearing_oring_25: geometry visual mesh filename=package://arena_robots/robots/rskomnidirectional/meshes/bea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
- link pin_bearing_oring_26: geometry visual mesh filename=package://arena_robots/robots/rskomnidirectional/meshes/bea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
- link pin_bearing_oring_27: geometry visual mesh filename=package://arena_robots/robots/rskomnidirectional/meshes/bea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
- link pin_bearing_oring_28: geometry visual mesh filename=package://arena_robots/robots/rskomnidirectional/meshes/bea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
- link pin_bearing_oring_29: geometry visual mesh filename=package://arena_robots/robots/rskomnidirectional/meshes/bea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
- link pin_bearing_oring_3: geometry visual mesh filename=package://arena_robots/robots/rskomnidirectional/meshes/bea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
- link pin_bearing_oring_30: geometry visual mesh filename=package://arena_robots/robots/rskomnidirectional/meshes/bea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
- link pin_bearing_oring_31: geometry visual mesh filename=package://arena_robots/robots/rskomnidirectional/meshes/bea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
- link pin_bearing_oring_32: geometry visual mesh filename=package://arena_robots/robots/rskomnidirectional/meshes/bea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
- link pin_bearing_oring_33: geometry visual mesh filename=package://arena_robots/robots/rskomnidirectional/meshes/bea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
- link pin_bearing_oring_34: geometry visual mesh filename=package://arena_robots/robots/rskomnidirectional/meshes/bea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
- link pin_bearing_oring_35: geometry visual mesh filename=package://arena_robots/robots/rskomnidirectional/meshes/bea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
- link pin_bearing_oring_36: geometry visual mesh filename=package://arena_robots/robots/rskomnidirectional/meshes/bea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
- link pin_bearing_oring_37: geometry visual mesh filename=package://arena_robots/robots/rskomnidirectional/meshes/bea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
- link pin_bearing_oring_38: geometry visual mesh filename=package://arena_robots/robots/rskomnidirectional/meshes/bea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
- link pin_bearing_oring_39: geometry visual mesh filename=package://arena_robots/robots/rskomnidirectional/meshes/bea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
- link pin_bearing_oring_4: geometry visual mesh filename=package://arena_robots/robots/rskomnidirectional/meshes/bea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
- link pin_bearing_oring_40: geometry visual mesh filename=package://arena_robots/robots/rskomnidirectional/meshes/bea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
- link pin_bearing_oring_41: geometry visual mesh filename=package://arena_robots/robots/rskomnidirectional/meshes/bea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
- link pin_bearing_oring_42: geometry visual mesh filename=package://arena_robots/robots/rskomnidirectional/meshes/bea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
- link pin_bearing_oring_43: geometry visual mesh filename=package://arena_robots/robots/rskomnidirectional/meshes/bea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
- link pin_bearing_oring_44: geometry visual mesh filename=package://arena_robots/robots/rskomnidirectional/meshes/bea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
- link pin_bearing_oring_45: geometry visual mesh filename=package://arena_robots/robots/rskomnidirectional/meshes/bea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
- link pin_bearing_oring_46: geometry visual mesh filename=package://arena_robots/robots/rskomnidirectional/meshes/bea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
- link pin_bearing_oring_47: geometry visual mesh filename=package://arena_robots/robots/rskomnidirectional/meshes/bea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
- link pin_bearing_oring_48: geometry visual mesh filename=package://arena_robots/robots/rskomnidirectional/meshes/bea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
- link pin_bearing_oring_49: geometry visual mesh filename=package://arena_robots/robots/rskomnidirectional/meshes/bea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
- link pin_bearing_oring_5: geometry visual mesh filename=package://arena_robots/robots/rskomnidirectional/meshes/bea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
- link pin_bearing_oring_50: geometry visual mesh filename=package://arena_robots/robots/rskomnidirectional/meshes/bea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
- link pin_bearing_oring_51: geometry visual mesh filename=package://arena_robots/robots/rskomnidirectional/meshes/bea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
- link pin_bearing_oring_52: geometry visual mesh filename=package://arena_robots/robots/rskomnidirectional/meshes/bea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
- link pin_bearing_oring_53: geometry visual mesh filename=package://arena_robots/robots/rskomnidirectional/meshes/bea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
- link pin_bearing_oring_54: geometry visual mesh filename=package://arena_robots/robots/rskomnidirectional/meshes/bea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
- link pin_bearing_oring_55: geometry visual mesh filename=package://arena_robots/robots/rskomnidirectional/meshes/bea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
- link pin_bearing_oring_56: geometry visual mesh filename=package://arena_robots/robots/rskomnidirectional/meshes/bea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
- link pin_bearing_oring_57: geometry visual mesh filename=package://arena_robots/robots/rskomnidirectional/meshes/bea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
- link pin_bearing_oring_58: geometry visual mesh filename=package://arena_robots/robots/rskomnidirectional/meshes/bea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
- link pin_bearing_oring_59: geometry visual mesh filename=package://arena_robots/robots/rskomnidirectional/meshes/bea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
- link pin_bearing_oring_6: geometry visual mesh filename=package://arena_robots/robots/rskomnidirectional/meshes/bea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
- link pin_bearing_oring_60: geometry visual mesh filename=package://arena_robots/robots/rskomnidirectional/meshes/bea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
- link pin_bearing_oring_7: geometry visual mesh filename=package://arena_robots/robots/rskomnidirectional/meshes/bea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
- link pin_bearing_oring_8: geometry visual mesh filename=package://arena_robots/robots/rskomnidirectional/meshes/bea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
- link pin_bearing_oring_9: geometry visual mesh filename=package://arena_robots/robots/rskomnidirectional/meshes/bea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
- link wheel_no_passives: geometry collision sphere radius=0.0345; visual mesh filename=package://arena_robots/robots/rskomnidirectional/meshes/cou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
- link wheel_no_passives_2: geometry collision sphere radius=0.0345; visual mesh filename=package://arena_robots/robots/rskomnidirectional/meshes/cou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
- link wheel_no_passives_3: geometry collision sphere radius=0.0345; visual mesh filename=package://arena_robots/robots/rskomnidirectional/meshes/cou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
Joints:
- joint imu_link_joint: origin xyz=0 0 0 rpy=0 0 0 -> xyz=0.0 0.0 0.0 rpy=0.0 0.0 0.0
- joint lidar_joint: origin xyz=0 0 0.3 rpy=0 0 0 -> xyz=0.0 0.0 0.3 rpy=0.0 0.0 0.0
- joint wheel1_passive_1: axis 0 0 1 -> (none); limit effort=10 velocity=10 -> (none); type continuous -> fixed
- joint wheel1_passive_10: axis 0 0 1 -> (none); limit effort=10 velocity=10 -> (none); type continuous -> fixed
- joint wheel1_passive_11: axis 0 0 1 -> (none); limit effort=10 velocity=10 -> (none); type continuous -> fixed
- joint wheel1_passive_12: axis 0 0 1 -> (none); limit effort=10 velocity=10 -> (none); type continuous -> fixed
- joint wheel1_passive_13: axis 0 0 1 -> (none); limit effort=10 velocity=10 -> (none); type continuous -> fixed
- joint wheel1_passive_14: axis 0 0 1 -> (none); limit effort=10 velocity=10 -> (none); type continuous -> fixed
- joint wheel1_passive_15: axis 0 0 1 -> (none); limit effort=10 velocity=10 -> (none); type continuous -> fixed
- joint wheel1_passive_16: axis 0 0 1 -> (none); limit effort=10 velocity=10 -> (none); type continuous -> fixed
- joint wheel1_passive_17: axis 0 0 1 -> (none); limit effort=10 velocity=10 -> (none); type continuous -> fixed
- joint wheel1_passive_18: axis 0 0 1 -> (none); limit effort=10 velocity=10 -> (none); type continuous -> fixed
- joint wheel1_passive_19: axis 0 0 1 -> (none); limit effort=10 velocity=10 -> (none); type continuous -> fixed
- joint wheel1_passive_2: axis 0 0 1 -> (none); limit effort=10 velocity=10 -> (none); type continuous -> fixed
- joint wheel1_passive_20: axis 0 0 1 -> (none); limit effort=10 velocity=10 -> (none); type continuous -> fixed
- joint wheel1_passive_3: axis 0 0 1 -> (none); limit effort=10 velocity=10 -> (none); type continuous -> fixed
- joint wheel1_passive_4: axis 0 0 1 -> (none); limit effort=10 velocity=10 -> (none); type continuous -> fixed
- joint wheel1_passive_5: axis 0 0 1 -> (none); limit effort=10 velocity=10 -> (none); type continuous -> fixed
- joint wheel1_passive_6: axis 0 0 1 -> (none); limit effort=10 velocity=10 -> (none); type continuous -> fixed
- joint wheel1_passive_7: axis 0 0 1 -> (none); limit effort=10 velocity=10 -> (none); type continuous -> fixed
- joint wheel1_passive_8: axis 0 0 1 -> (none); limit effort=10 velocity=10 -> (none); type continuous -> fixed
- joint wheel1_passive_9: axis 0 0 1 -> (none); limit effort=10 velocity=10 -> (none); type continuous -> fixed
- joint wheel2_passive1: axis 0 0 1 -> (none); limit effort=10 velocity=10 -> (none); type continuous -> fixed
- joint wheel2_passive10: axis 0 0 1 -> (none); limit effort=10 velocity=10 -> (none); type continuous -> fixed
- joint wheel2_passive11: axis 0 0 1 -> (none); limit effort=10 velocity=10 -> (none); type continuous -> fixed
- joint wheel2_passive12: axis 0 0 1 -> (none); limit effort=10 velocity=10 -> (none); type continuous -> fixed
- joint wheel2_passive13: axis 0 0 1 -> (none); limit effort=10 velocity=10 -> (none); type continuous -> fixed
- joint wheel2_passive14: axis 0 0 1 -> (none); limit effort=10 velocity=10 -> (none); type continuous -> fixed
- joint wheel2_passive15: axis 0 0 1 -> (none); limit effort=10 velocity=10 -> (none); type continuous -> fixed
- joint wheel2_passive16: axis 0 0 1 -> (none); limit effort=10 velocity=10 -> (none); type continuous -> fixed
- joint wheel2_passive17: axis 0 0 1 -> (none); limit effort=10 velocity=10 -> (none); type continuous -> fixed
- joint wheel2_passive18: axis 0 0 1 -> (none); limit effort=10 velocity=10 -> (none); type continuous -> fixed
- joint wheel2_passive19: axis 0 0 1 -> (none); limit effort=10 velocity=10 -> (none); type continuous -> fixed
- joint wheel2_passive2: axis 0 0 1 -> (none); limit effort=10 velocity=10 -> (none); type continuous -> fixed
- joint wheel2_passive20: axis 0 0 1 -> (none); limit effort=10 velocity=10 -> (none); type continuous -> fixed
- joint wheel2_passive3: axis 0 0 1 -> (none); limit effort=10 velocity=10 -> (none); type continuous -> fixed
- joint wheel2_passive4: axis 0 0 1 -> (none); limit effort=10 velocity=10 -> (none); type continuous -> fixed
- joint wheel2_passive5: axis 0 0 1 -> (none); limit effort=10 velocity=10 -> (none); type continuous -> fixed
- joint wheel2_passive6: axis 0 0 1 -> (none); limit effort=10 velocity=10 -> (none); type continuous -> fixed
- joint wheel2_passive7: axis 0 0 1 -> (none); limit effort=10 velocity=10 -> (none); type continuous -> fixed
- joint wheel2_passive8: axis 0 0 1 -> (none); limit effort=10 velocity=10 -> (none); type continuous -> fixed
- joint wheel2_passive9: axis 0 0 1 -> (none); limit effort=10 velocity=10 -> (none); type continuous -> fixed
- joint wheel3_passive1: axis 0 0 1 -> (none); limit effort=10 velocity=10 -> (none); type continuous -> fixed
- joint wheel3_passive10: axis 0 0 1 -> (none); limit effort=10 velocity=10 -> (none); type continuous -> fixed
- joint wheel3_passive11: axis 0 0 1 -> (none); limit effort=10 velocity=10 -> (none); type continuous -> fixed
- joint wheel3_passive12: axis 0 0 1 -> (none); limit effort=10 velocity=10 -> (none); type continuous -> fixed
- joint wheel3_passive13: axis 0 0 1 -> (none); limit effort=10 velocity=10 -> (none); type continuous -> fixed
- joint wheel3_passive14: axis 0 0 1 -> (none); limit effort=10 velocity=10 -> (none); type continuous -> fixed
- joint wheel3_passive15: axis 0 0 1 -> (none); limit effort=10 velocity=10 -> (none); type continuous -> fixed
- joint wheel3_passive16: axis 0 0 1 -> (none); limit effort=10 velocity=10 -> (none); type continuous -> fixed
- joint wheel3_passive17: axis 0 0 1 -> (none); limit effort=10 velocity=10 -> (none); type continuous -> fixed
- joint wheel3_passive18: axis 0 0 1 -> (none); limit effort=10 velocity=10 -> (none); type continuous -> fixed
- joint wheel3_passive19: axis 0 0 1 -> (none); limit effort=10 velocity=10 -> (none); type continuous -> fixed
- joint wheel3_passive2: axis 0 0 1 -> (none); limit effort=10 velocity=10 -> (none); type continuous -> fixed
- joint wheel3_passive20: axis 0 0 1 -> (none); limit effort=10 velocity=10 -> (none); type continuous -> fixed
- joint wheel3_passive3: axis 0 0 1 -> (none); limit effort=10 velocity=10 -> (none); type continuous -> fixed
- joint wheel3_passive4: axis 0 0 1 -> (none); limit effort=10 velocity=10 -> (none); type continuous -> fixed
- joint wheel3_passive5: axis 0 0 1 -> (none); limit effort=10 velocity=10 -> (none); type continuous -> fixed
- joint wheel3_passive6: axis 0 0 1 -> (none); limit effort=10 velocity=10 -> (none); type continuous -> fixed
- joint wheel3_passive7: axis 0 0 1 -> (none); limit effort=10 velocity=10 -> (none); type continuous -> fixed
- joint wheel3_passive8: axis 0 0 1 -> (none); limit effort=10 velocity=10 -> (none); type continuous -> fixed
- joint wheel3_passive9: axis 0 0 1 -> (none); limit effort=10 velocity=10 -> (none); type continuous -> fixed
