Commit message: fix mpo700 chassis collision resting below wheels

File: arena_robots/robots/mpo700/urdf/xacros/mpo_700_body.urdf.xacro (robot description, xacro)
@@ -23,7 +23,7 @@
       </visual>
       <collision>
-        <origin rpy="0 0 -1.571" xyz="0. 0. 0."/>
+        <origin rpy="0 0 0" xyz="-0.01 0. 0.255"/>
         <geometry>
-          <mesh filename="package://arena_robots/robots/mpo700/meshes/MPO-700-BODY.dae" scale="0.001 0.001 0.001"/>
+          <box size="0.63 0.506 0.19"/>
         </geometry>
       </collision>
