Commit message: oakd_rgbd start

File: arena_robots/components/camera/oakd_rgbd/oakd_rgb.urdf.xacro (robot description, xacro)
@@ -1,3 +1,197 @@
 <?xml version="1.0"?>
-<robot name="oakd_rgb" xlmns:xacro="https://wiki.ros.org/xacro">
+<robot xmlns:xacro="http://ros.org/wiki/xacro">
+<xacro:macro name="oakd" params="name:=oakd parent_link *origin model:=pro">
+  <xacro:include filename="$(find irobot_create_description)/urdf/common_properties.urdf.xacro"/>
+  <xacro:include filename="$(find arena_robots)/urdf/gz_rgbd_camera.xacro"/>
+  <xacro:property name="mass"       value="0.061"/>
+  <xacro:property name="baseline" value="0.075" />
+  <xacro:property name="M_PI"     value="3.1415926535897931" />
+  <xacro:property name="collision_length_x"   value="${2.25*cm2m}" />
+  <xacro:property name="collision_length_y"   value="${9.7*cm2m}" />
+  <xacro:property name="collision_length_z"   value="${3*cm2m}" />
+  <xacro:property name="collision_offset_x"   value="${-1.1*cm2m}" />
+  <xacro:property name="collision_offset_y"   value="${0*cm2m}" />
+  <xacro:property name="collision_offset_z"   value="${-0.5*cm2m}" />
+  <xacro:property name="base_frame" value="${name}_link"/>
+  <!-- Base frame -->
+  <joint name="${name}_joint" type="fixed">
+    <parent link="${parent_link}"/>
+    <child link="${base_frame}"/>
+    <xacro:insert_block name="origin"/>
+  </joint>
+  <link name="${base_frame}">
+    <visual>
+      <geometry>
+        <mesh filename="package://turtlebot4_description/meshes/${name}_${model}.dae" scale="1 1 1" />
+      </geometry>
+    </visual>
+    <collision>
+      <origin xyz="${collision_offset_x} ${collision_offset_y} ${collision_offset_z}"/>
+      <geometry>
+        <box size="${collision_length_x} ${collision_length_y} ${collision_length_z}"/>
+      </geometry>
+    </collision>
+    <inertial>
+      <mass value="${mass}"/>
+      <inertia ixx="0.00000202475" ixy="0.0" ixz="0.0"
+	             iyy="0.00001527320" iyz="0.0" izz="0.00001605536" />
+    </inertial>
+  </link>
+  <!-- RGB Camera -->
+  <link name="${name}_rgb_camera_frame">
+    <xacro:inertial_dummy/>
+  </link>
+  <joint name="${name}_rgb_camera_joint" type="fixed">
+      <parent link="${base_frame}"/>
+      <child link="${name}_rgb_camera_frame"/>
+      <origin xyz="0 0 0" rpy="0 0 0" />
+  </joint>
+  <link name="${name}_rgb_camera_optical_frame">
+    <xacro:inertial_dummy/>
+  </link>
+  <joint name="${name}_rgb_camera_optical_joint" type="fixed">
+      <origin xyz="0 0 0" rpy="-${M_PI/2} 0.0 -${M_PI/2}"/>
+      <parent link="${name}_rgb_camera_frame"/>
+      <child link="${name}_rgb_camera_optical_frame"/>
+  </joint>
+  <!-- Left Camera -->
+  <link name="${name}_left_camera_frame">
+    <xacro:inertial_dummy/>
+  </link>
+  <joint name="${name}_left_camera_joint" type="fixed">
+      <parent link="${base_frame}"/>
+      <child link="${name}_left_camera_frame"/>
+      <origin xyz="0 ${baseline/2} 0" rpy="0 0 0" />
+  </joint>
+  <link name="${name}_left_camera_optical_frame">
+    <xacro:inertial_dummy/>
+  </link>
+  <joint name="${name}_left_camera_optical_joint" type="fixed">
+      <origin xyz="0 0 0" rpy="-${M_PI/2} 0.0 -${M_PI/2}"/>
+      <parent link="${name}_left_camera_frame"/>
+      <child link="${name}_left_camera_optical_frame"/>
+  </joint>
+  <!-- Right Camera -->
+  <link name="${name}_right_camera_frame">
+    <xacro:inertial_dummy/>
+  </link>
+  <joint name="${name}_right_camera_joint" type="fixed">
+      <parent link="${base_frame}"/>
+      <child link="${name}_right_camera_frame"/>
+      <origin xyz="0 -${baseline/2} 0" rpy="0 0 0" />
+  </joint>
+  <link name="${name}_right_camera_optical_frame">
+    <xacro:inertial_dummy/>
+  </link>
+  <joint name="${name}_right_camera_optical_joint" type="fixed">
+      <origin xyz="0 0 0" rpy="-${M_PI/2} 0.0 -${M_PI/2}"/>
+      <parent link="${name}_right_camera_frame"/>
+      <child link="${name}_right_camera_optical_frame"/>
+  </joint>
+  <!-- IMU -->
+  <link name="${name}_imu_frame">
+    <xacro:inertial_dummy/>
+  </link>
+  <joint name="${name}_imu_joint" type="fixed">
+      <parent link="${base_frame}"/>
+      <child link="${name}_imu_frame"/>
+      <origin xyz="0 0 0" rpy="-${M_PI/2} 0 -${M_PI/2}" />
+  </joint>
+  <gazebo reference="${name}_imu_joint">
+    <sensor name="imu_sensor" type="imu">
+      <plugin filename="libgz-sim-imu-system" name="gz::sim::systems::Imu">
+        <topic>/imu/data</topic>
+        <frame_id>${name}_imu_frame</frame_id>
+      </plugin>
+      <always_on>true</always_on>
+      <update_rate>100</update_rate>
+      <visualize>true</visualize>
+      <imu>
+        <angular_velocity>
+          <x>
+            <noise type="gaussian">
+              <mean>0.0</mean>
+              <stddev>2e-4</stddev>
+              <bias_mean>0.0000075</bias_mean>
+              <bias_stddev>0.0000008</bias_stddev>
+            </noise>
+          </x>
+          <y>
+            <noise type="gaussian">
+              <mean>0.0</mean>
+              <stddev>2e-4</stddev>
+              <bias_mean>0.0000075</bias_mean>
+              <bias_stddev>0.0000008</bias_stddev>
+            </noise>
+          </y>
+          <z>
+            <noise type="gaussian">
+              <mean>0.0</mean>
+              <stddev>2e-4</stddev>
+              <bias_mean>0.0000075</bias_mean>
+              <bias_stddev>0.0000008</bias_stddev>
+            </noise>
+          </z>
+        </angular_velocity>
+        <linear_acceleration>
+          <x>
+            <noise type="gaussian">
+              <mean>0.0</mean>
+              <stddev>1.7e-2</stddev>
+              <bias_mean>0.1</bias_mean>
+              <bias_stddev>0.001</bias_stddev>
+            </noise>
+          </x>
+          <y>
+            <noise type="gaussian">
+              <mean>0.0</mean>
+              <stddev>1.7e-2</stddev>
+              <bias_mean>0.1</bias_mean>
+              <bias_stddev>0.001</bias_stddev>
+            </noise>
+          </y>
+          <z>
+            <noise type="gaussian">
+              <mean>0.0</mean>
+              <stddev>1.7e-2</stddev>
+              <bias_mean>0.1</bias_mean>
+              <bias_stddev>0.001</bias_stddev>
+            </noise>
+          </z>
+        </linear_acceleration>
+      </imu>
+    </sensor>
+    <material>Gazebo/Grey</material>
+  </gazebo>
+  <!-- Gazebo links and joints -->
+  <xacro:gz_rgbd_camera frame="${name}_rgb_camera_frame" sensor_name="rgbd_camera"
+                        fov="1.25" width="320" height="240" near="0.3" far="100" update_rate="30"/>
+  <gazebo reference="${name}_rgb_camera_frame">
+    <xacro:material_darkgray/>
+  </gazebo>
+  <gazebo reference="${name}_joint">
+    <preserveFixedJoint>true</preserveFixedJoint>
+  </gazebo>
+  <gazebo reference="${name}_rgb_camera_joint">
+    <preserveFixedJoint>true</preserveFixedJoint>
+  </gazebo>
+  <gazebo reference="${name}_rgb_camera_optical_joint">
+    <preserveFixedJoint>true</preserveFixedJoint>
+  </gazebo>
+  <gazebo reference="${name}_left_camera_joint">
+    <preserveFixedJoint>true</preserveFixedJoint>
+  </gazebo>
+  <gazebo reference="${name}_left_camera_optical_joint">
+    <preserveFixedJoint>true</preserveFixedJoint>
+  </gazebo>
+  <gazebo reference="${name}_right_camera_joint">
+    <preserveFixedJoint>true</preserveFixedJoint>
+  </gazebo>
+  <gazebo reference="${name}_right_camera_optical_joint">
+    <preserveFixedJoint>true</preserveFixedJoint>
+  </gazebo>
+  <gazebo reference="${name}_imu_joint">
+    <preserveFixedJoint>true</preserveFixedJoint>
+  </gazebo>
+</xacro:macro>
 </robot>

Commit message: add component meshes as submodules

File: arena_robots/components/camera/oakd_rgbd/oakd_rgb.urdf.xacro (robot description, xacro)
@@ -23,5 +23,5 @@
     <visual>
       <geometry>
-        <mesh filename="package://turtlebot4_description/meshes/${name}_${model}.dae" scale="1 1 1" />
+        <mesh filename="package://arena_robots/components/camera/oakd_rgbd/meshes/${name}_${model}.dae" scale="1 1 1" />
       </geometry>
     </visual>

File: arena_robots/components/imu/vectornav/vectornav.urdf.xacro (robot description, xacro)
@@ -28,5 +28,5 @@
         </material>
         <geometry>
-          <mesh filename="package://arena_robots/robots/rbvogui/meshes/imu/vectornav_vn100.stl"/>
+          <mesh filename="package://arena_robots/components/imu/vectornav/meshes/vectornav_vn100.stl"/>
         </geometry>
       </visual>

File: arena_robots/components/lidar/hokuyo_ust20lx/hokuyo_ust20lx.urdf.xacro (robot description, xacro)
@@ -32,5 +32,5 @@
         <origin xyz="0 0 0" rpy="0 0 0"/>
         <geometry>
-          <mesh filename="package://arena_robots/robots/rbvogui/meshes/hokuyo_ust_20lx.dae"/>
+          <mesh filename="package://arena_robots/components/lidar/hokuyo_ust20lx/meshes/hokuyo_ust_20lx.dae"/>
         </geometry>
       </visual>

File: arena_robots/components/lidar/robosense_helios_16p/robosense_helios_16p.urdf.xacro (robot description, xacro)
@@ -25,5 +25,5 @@
         <origin xyz="0 0 0" rpy="0 0 0"/>
         <geometry>
-          <mesh filename="package://arena_robots/robots/rbvogui/meshes/3d_lidar/robotsense/helios_16p.stl"/>
+          <mesh filename="package://arena_robots/components/lidar/robosense_helios_16p/meshes/helios_16p.stl"/>
         </geometry>
       </collision>
@@ -31,5 +31,5 @@
         <origin xyz="0 0 0" rpy="0 0 0"/>
         <geometry>
-          <mesh filename="package://arena_robots/robots/rbvogui/meshes/3d_lidar/robotsense/helios_16p.stl"/>
+          <mesh filename="package://arena_robots/components/lidar/robosense_helios_16p/meshes/helios_16p.stl"/>
         </geometry>
         <material name="blackgray_color">

File: arena_robots/components/lidar/rplidar/rplidar.urdf.xacro (robot description, xacro)
@@ -26,5 +26,5 @@
     <visual>
       <geometry>
-        <mesh filename="package://turtlebot4_description/meshes/rplidar.dae" scale="1 1 1" />
+        <mesh filename="package://arena_robots/lidar/rplidar/meshes/rplidar.dae" scale="1 1 1" />
       </geometry>
     </visual>

File: arena_robots/components/lidar/sick_microscan3/sick_microscan3.urdf.xacro (robot description, xacro)
@@ -26,5 +26,5 @@
         <origin xyz="0 0 0" rpy="0 0 0"/>
         <geometry>
-		  <mesh filename="package://arena_robots/robots/rbrobout/meshes/2d_lidar/sick/microscan3.dae"/>
+		  <mesh filename="package://arena_robots/components/lidar/sick_microscan3/meshes/microscan3.dae"/>
         </geometry>
       </visual>
@@ -32,5 +32,5 @@
         <origin xyz="0 0 0" rpy="0 0 0"/>
         <geometry>
-		  <mesh filename="package://arena_robots/robots/rbrobout/meshes/2d_lidar/sick/microscan3.dae"/>
+		  <mesh filename="package://arena_robots/components/lidar/sick_microscan3/meshes/microscan3.dae"/>
         </geometry>
       </collision>

File: arena_robots/components/lidar/sick_s300/sick_s300.urdf.xacro (robot description, xacro)
@@ -28,5 +28,5 @@
         <origin xyz="0 0 0" rpy="${-pi/2} 0 0"/>
         <geometry>
-          <mesh filename="package://arena_robots/robots/rbvogui/meshes/2d_lidar/sick/s300.dae"/>
+          <mesh filename="package://arena_robots/components/lidar/sick_s300/meshes/s300.dae"/>
         </geometry>
       </visual>
@@ -34,5 +34,5 @@
         <origin xyz="0 0 0" rpy="${-pi/2} 0 0"/>
         <geometry>
-          <mesh filename="package://arena_robots/robots/rbvogui/meshes/2d_lidar/sick/s300.dae"/>
+          <mesh filename="package://arena_robots/components/lidar/sick_s300/meshes/s300.dae"/>
         </geometry>
       </collision>
