Commit message: fix: update hokuyo submodule url, add create dependency, fix rplidar mesh path

File: arena_robots/components/lidar/rplidar/rplidar.urdf.xacro (robot description, xacro)
@@ -26,5 +26,5 @@
     <visual>
       <geometry>
-        <mesh filename="package://arena_robots/lidar/rplidar/meshes/rplidar.dae" scale="1 1 1" />
+        <mesh filename="package://arena_robots/components/lidar/rplidar/meshes/rplidar.dae" scale="1 1 1" />
       </geometry>
     </visual>
