Commit message: update d435 goldens

File: arena_robots/tests/golden/rbkairos_default.urdf (robot description, URDF)
Before this commit: robot rbkairos, 32 links, 31 joints
Links:
- removed link robot_front_rgbd_camera_base_link
- added link robot_front_rgbd_camera_bottom_screw_frame
Joints:
- removed joint robot_front_rgbd_camera_base_joint
- added joint robot_front_rgbd_camera_link_joint: type fixed, parent robot_front_rgbd_camera_bottom_screw_frame, child robot_front_rgbd_camera_link, origin xyz=0.0106 0.0175 0.0125 rpy=0 0 0
- joint robot_front_rgbd_camera_joint: child robot_front_rgbd_camera_link -> robot_front_rgbd_camera_bottom_screw_frame; origin xyz=0.01 0.02 0 rpy=0 0 0 -> xyz=0.3585 0.0 0.25062 rpy=0 0 0; parent robot_front_rgbd_camera_base_link -> robot_base_link

File: arena_robots/tests/golden/rbsummit_default.urdf (robot description, URDF)
Before this commit: robot summit_xl, 23 links, 22 joints
Links:
- removed link robot_front_rgbd_camera_base_link
- added link robot_front_rgbd_camera_bottom_screw_frame
Joints:
- removed joint robot_front_rgbd_camera_base_joint
- added joint robot_front_rgbd_camera_link_joint: type fixed, parent robot_front_rgbd_camera_bottom_screw_frame, child robot_front_rgbd_camera_link, origin xyz=0.0106 0.0175 0.0125 rpy=0 0 0
- joint robot_front_rgbd_camera_joint: child robot_front_rgbd_camera_link -> robot_front_rgbd_camera_bottom_screw_frame; origin xyz=0.01 0.02 0 rpy=0 0 0 -> xyz=0.324 0.012 0.172 rpy=0 0 0; parent robot_front_rgbd_camera_base_link -> robot_base_link

File: arena_robots/tests/golden/rbtheron_default.urdf (robot description, URDF)
Before this commit: robot rb_theron, 45 links, 44 joints
Links:
- removed link robot_front_rgbd_camera_base_link
- removed link robot_rear_rgbd_camera_base_link
- added link robot_front_rgbd_camera_bottom_screw_frame
- added link robot_rear_rgbd_camera_bottom_screw_frame
Joints:
- removed joint robot_front_rgbd_camera_base_joint
- removed joint robot_rear_rgbd_camera_base_joint
- added joint robot_front_rgbd_camera_link_joint: type fixed, parent robot_front_rgbd_camera_bottom_screw_frame, child robot_front_rgbd_camera_link, origin xyz=0.0106 0.0175 0.0125 rpy=0 0 0
- added joint robot_rear_rgbd_camera_link_joint: type fixed, parent robot_rear_rgbd_camera_bottom_screw_frame, child robot_rear_rgbd_camera_link, origin xyz=0.0106 0.0175 0.0125 rpy=0 0 0
- joint robot_front_rgbd_camera_joint: child robot_front_rgbd_camera_link -> robot_front_rgbd_camera_bottom_screw_frame; origin xyz=0.01 0.02 0 rpy=0 0 0 -> xyz=0.3045 0.0 0.1898 rpy=0 0 0; parent robot_front_rgbd_camera_base_link -> robot_base_link
- joint robot_rear_rgbd_camera_joint: child robot_rear_rgbd_camera_link -> robot_rear_rgbd_camera_bottom_screw_frame; origin xyz=0.01 0.02 0 rpy=0 0 0 -> xyz=-0.3045 0.0 0.1158 rpy=0 0 3.141592653589793; parent robot_rear_rgbd_camera_base_link -> robot_base_link

File: arena_robots/tests/golden/rbvogui_default.urdf (robot description, URDF)
Before this commit: robot rbvogui, 41 links, 40 joints
Links:
- removed link robot_front_rgbd_camera_base_link
- removed link robot_rear_rgbd_camera_base_link
- added link robot_front_rgbd_camera_bottom_screw_frame
- added link robot_rear_rgbd_camera_bottom_screw_frame
Joints:
- removed joint robot_front_rgbd_camera_base_joint
- removed joint robot_rear_rgbd_camera_base_joint
- added joint robot_front_rgbd_camera_link_joint: type fixed, parent robot_front_rgbd_camera_bottom_screw_frame, child robot_front_rgbd_camera_link, origin xyz=0.0106 0.0175 0.0125 rpy=0 0 0
- added joint robot_rear_rgbd_camera_link_joint: type fixed, parent robot_rear_rgbd_camera_bottom_screw_frame, child robot_rear_rgbd_camera_link, origin xyz=0.0106 0.0175 0.0125 rpy=0 0 0
- joint robot_front_rgbd_camera_joint: child robot_front_rgbd_camera_link -> robot_front_rgbd_camera_bottom_screw_frame; origin xyz=0.01 0.02 0 rpy=0 0 0 -> xyz=0.46462 0.0 0.18258 rpy=0 0 0; parent robot_front_rgbd_camera_base_link -> robot_base_link
- joint robot_rear_rgbd_camera_joint: child robot_rear_rgbd_camera_link -> robot_rear_rgbd_camera_bottom_screw_frame; origin xyz=0.01 0.02 0 rpy=0 0 0 -> xyz=-0.503 0.0 0.29 rpy=0 0 -3.14159265359; parent robot_rear_rgbd_camera_base_link -> robot_base_link
