Commit message: model params and golden follow the camera defaults

File: arena_robots/tests/golden/turtlebot_default.urdf (robot description, URDF)
Before this commit: robot turtlebot, 49 links, 48 joints
Links:
- link oakd_link: geometry collision box size=0.0225 0.09699999999999999 0.03; visual mesh filename=package://arena_robots/components/camera/oakd_rgbd/meshes/o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 scale=1 1 1
- link rplidar_link: geometry collision box size=0.071 0.1 0.06; visual mesh filename=package://arena_robots/components/lidar/rplidar/meshes/rpli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 scale=1 1 1
Joints:
- joint oakd_joint: origin xyz=0.0584 0.0 0.09676 -> xyz=0.0584 0.0 0.09676 rpy=0.0 0.0 0.0
- joint rplidar_joint: origin xyz=-0.04 0.0 0.098715 rpy=0 0 1.5707963267948966 -> xyz=-0.04 0.0 0.098715 rpy=0.0 0.0 1.5707963267948966
