Commit message: hokuyo ust-20lx caps mirror the datasheet

File: arena_robots/tests/golden/rbtheron_default.urdf (robot description, URDF)
Before this commit: robot rb_theron, 45 links, 44 joints
Links:
- link robot_front_laser_base_link: geometry collision cylinder length=0.072 radius=0.022; visual mesh filename=package://arena_robots/components/lidar/hokuyo_ust20lx/mesh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
- link robot_front_rgbd_camera_link: mass 0.1 -> 0.072; geometry collision box size=0.02505 0.09 0.025; visual mesh filename=package://realsense2_description/meshes/d435.dae
- link robot_rear_laser_base_link: geometry collision cylinder length=0.072 radius=0.022; visual mesh filename=package://arena_robots/components/lidar/hokuyo_ust20lx/mesh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
- link robot_rear_rgbd_camera_link: mass 0.1 -> 0.072; geometry collision box size=0.02505 0.09 0.025; visual mesh filename=package://realsense2_description/meshes/d435.dae
- link robot_vectornav_base_link: geometry collision box size=0.036 0.037 0.009; visual mesh filename=package://arena_robots/components/imu/vectornav/meshes/vect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
Joints:
- joint robot_front_laser_base_joint: origin xyz=0.2675 -0.215 0.1613 rpy=0 -3.141592653589793 2.356194490192345 -> xyz=0.2675 -0.215 0.1613 rpy=0.0 -3.141592653589793 2.356194490192345
- joint robot_front_rgbd_camera_joint: origin xyz=0.3045 0.0 0.1898 rpy=0 0 0 -> xyz=0.3045 0.0 0.1898 rpy=0.0 0.0 0.0
- joint robot_front_rgbd_camera_link_joint: origin xyz=0.0106 0.0175 0.0125 rpy=0 0 0 -> xyz=0.010600000000000002 0.0175 0.0125 rpy=0 0 0
- joint robot_rear_laser_base_joint: origin xyz=-0.2675 0.215 0.1613 rpy=0 -3.141592653589793 -0.7853981633974483 -> xyz=-0.2675 0.215 0.1613 rpy=0.0 -3.141592653589793 -0.7853981633974483
- joint robot_rear_rgbd_camera_joint: origin xyz=-0.3045 0.0 0.1158 rpy=0 0 3.141592653589793 -> xyz=-0.3045 0.0 0.1158 rpy=0.0 0.0 3.141592653589793
- joint robot_rear_rgbd_camera_link_joint: origin xyz=0.0106 0.0175 0.0125 rpy=0 0 0 -> xyz=0.010600000000000002 0.0175 0.0125 rpy=0 0 0
- joint robot_vectornav_base_joint: origin xyz=-0.1975 0.0 0.1598 rpy=0 0 0 -> xyz=-0.1975 0.0 0.1598 rpy=0.0 0.0 0.0
