Commit message: telemetry

File: arena_robots/robots/jackal/urdf/jackal.urdf.xacro (robot description, xacro)
@@ -32,7 +32,7 @@
       </visual>
       <collision>
-        <origin xyz="0 0 0" rpy="${PI/2} 0 0"/>
-        <geometry>
-          <cylinder radius="${wheel_radius}" length="${wheel_width}"/>
+        <origin xyz="0 0 0" rpy="0 0 0"/>
+        <geometry>
+          <sphere radius="${wheel_radius}"/>
         </geometry>
       </collision>
@@ -220,5 +220,6 @@
        of these into the final description is controlled by optenv variables, which
        default each one to off.-->
-  <xacro:include filename="$(find jackal_description)/urdf/accessories.urdf.xacro" />
+  <!-- Bring in simulation accessories for everything in accessories.urdf.xacro -->
+  <!-- <xacro:include filename="$(find jackal_description)/urdf/accessories.urdf.xacro" /> -->
   <!-- Optional custom includes. -->
   <xacro:include filename="$(optenv JACKAL_URDF_EXTRAS empty.urdf)" />
