Commit message: sick s300 mirrors the datasheet

File: arena_robots/components/lidar/sick_s300/sick_s300.urdf.xacro (robot description, xacro)
@@ -13,6 +13,6 @@
                        topic_prefix:=~/
                        gpu:=false
-                       min_angle:=${-radians(130)}
-                       max_angle:=${radians(130)}">
+                       min_angle:=${-radians(135)}
+                       max_angle:=${radians(135)}">
     <!-- node_namespace is used from node_name if not set -->
     <xacro:if value="${node_namespace == None}">
@@ -55,5 +55,5 @@
       gazebo_ignition="${gazebo_ignition}"
       min_range="0.05"
-      max_range="10.0"
+      max_range="30.0"
       min_angle="${min_angle}"
       max_angle="${max_angle}"
@@ -61,5 +61,5 @@
       rate="25.0"
       resolution="0.00575"
-      samples="270"
+      samples="541"
     >
     </xacro:lidar_2d_plugin>

File: arena_robots/tests/golden/mpo700_default.urdf (robot description, URDF)
Before this commit: robot mpo700, 14 links, 13 joints
Links:
- link base_footprint: geometry collision box size=0.63 0.506 0.19; visual mesh filename=package://arena_robots/robots/mpo700/meshes/MPO-700-BODY.dae scale=0.001 0.001 0.001
- link front_laser_base_link: geometry collision mesh filename=package://arena_robots/components/lidar/sick_s300/meshes/s3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; visual mesh filename=package://arena_robots/components/lidar/sick_s300/meshes/s3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
- link rear_laser_base_link: geometry collision mesh filename=package://arena_robots/components/lidar/sick_s300/meshes/s3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; visual mesh filename=package://arena_robots/components/lidar/sick_s300/meshes/s3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
Joints:
- joint front_laser_base_joint: origin xyz=0.338 0.288 0.223 rpy=3.14 0 0.79 -> xyz=0.338 0.288 0.223 rpy=3.14 0.0 0.79
- joint rear_laser_base_joint: origin xyz=-0.338 -0.288 0.223 rpy=3.14 0 3.93 -> xyz=-0.338 -0.288 0.223 rpy=3.14 0.0 3.93

File: arena_robots/tests/golden/rbkairos_default.urdf (robot description, URDF)
Before this commit: robot rbkairos, 32 links, 31 joints
Links:
- link robot_front_laser_base_link: geometry collision mesh filename=package://arena_robots/components/lidar/sick_s300/meshes/s3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; visual mesh filename=package://arena_robots/components/lidar/sick_s300/meshes/s3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
- link robot_front_rgbd_camera_link: mass 0.1 -> 0.072; geometry collision box size=0.02505 0.09 0.025; visual mesh filename=package://realsense2_description/meshes/d435.dae
- link robot_rear_laser_base_link: geometry collision mesh filename=package://arena_robots/components/lidar/sick_s300/meshes/s3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; visual mesh filename=package://arena_robots/components/lidar/sick_s300/meshes/s3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
- link robot_vectornav_base_link: geometry collision box size=0.036 0.037 0.009; visual mesh filename=package://arena_robots/components/imu/vectornav/meshes/vect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
Joints:
- joint robot_front_laser_base_joint: origin xyz=0.42109 -0.32737 0.16037 rpy=0 -3.14159265359 2.3561944901925003 -> xyz=0.42109 -0.32737 0.16037 rpy=0.0 -3.141592653589793 2.356194490192345
- joint robot_front_rgbd_camera_joint: origin xyz=0.3585 0.0 0.25062 rpy=0 0 0 -> xyz=0.3585 0.0 0.25062 rpy=0.0 0.0 0.0
- joint robot_front_rgbd_camera_link_joint: origin xyz=0.0106 0.0175 0.0125 rpy=0 0 0 -> xyz=0.010600000000000002 0.0175 0.0125 rpy=0 0 0
- joint robot_rear_laser_base_joint: origin xyz=-0.42109 0.32737 0.16037 rpy=0 -3.14159265359 -0.7853981633975 -> xyz=-0.42109 0.32737 0.16037 rpy=0.0 -3.141592653589793 -0.7853981633974483
- joint robot_vectornav_base_joint: origin xyz=0.127 -0.129 0.212 rpy=0 0 0 -> xyz=0.127 -0.129 0.212 rpy=0.0 0.0 0.0

File: arena_robots/tests/golden/rbvogui_default.urdf (robot description, URDF)
Before this commit: robot rbvogui, 41 links, 40 joints
Links:
- link robot_front_laser_base_link: geometry collision mesh filename=package://arena_robots/components/lidar/sick_s300/meshes/s3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; visual mesh filename=package://arena_robots/components/lidar/sick_s300/meshes/s3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
- link robot_front_rgbd_camera_link: mass 0.1 -> 0.072; geometry collision box size=0.02505 0.09 0.025; visual mesh filename=package://realsense2_description/meshes/d435.dae
- link robot_rear_laser_base_link: geometry collision mesh filename=package://arena_robots/components/lidar/sick_s300/meshes/s3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; visual mesh filename=package://arena_robots/components/lidar/sick_s300/meshes/s3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
- link robot_rear_rgbd_camera_link: mass 0.1 -> 0.072; geometry collision box size=0.02505 0.09 0.025; visual mesh filename=package://realsense2_description/meshes/d435.dae
- link robot_vectornav_base_link: geometry collision box size=0.036 0.037 0.009; visual mesh filename=package://arena_robots/components/imu/vectornav/meshes/vect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
Joints:
- joint robot_front_laser_base_joint: origin xyz=0.53 0.33 0.1145 rpy=3.14159265359 0 0.7853981633975 -> xyz=0.53 0.33 0.1145 rpy=3.141592653589793 0.0 0.7853981633974483
- joint robot_front_rgbd_camera_joint: origin xyz=0.46462 0.0 0.18258 rpy=0 0 0 -> xyz=0.46462 0.0 0.18258 rpy=0.0 0.0 0.0
- joint robot_front_rgbd_camera_link_joint: origin xyz=0.0106 0.0175 0.0125 rpy=0 0 0 -> xyz=0.010600000000000002 0.0175 0.0125 rpy=0 0 0
- joint robot_rear_laser_base_joint: origin xyz=-0.53 -0.33 0.1145 rpy=3.14159265359 0 -2.3561944901925003 -> xyz=-0.53 -0.33 0.1145 rpy=3.141592653589793 0.0 -2.356194490192345
- joint robot_rear_rgbd_camera_joint: origin xyz=-0.503 0.0 0.29 rpy=0 0 -3.14159265359 -> xyz=-0.503 0.0 0.29 rpy=0.0 0.0 -3.141592653589793
- joint robot_rear_rgbd_camera_link_joint: origin xyz=0.0106 0.0175 0.0125 rpy=0 0 0 -> xyz=0.010600000000000002 0.0175 0.0125 rpy=0 0 0
- joint robot_vectornav_base_joint: origin xyz=0.3 -0.3 0.0725 rpy=0 0 0 -> xyz=0.3 -0.3 0.0725 rpy=0.0 0.0 0.0
