Commit message: boxer lidars mirror the datasheets

File: arena_robots/components/lidar/boxer_front/lidar.urdf.xacro (robot description, xacro)
@@ -36,5 +36,5 @@
           <scan>
             <horizontal>
-              <samples>720</samples>
+              <samples>2161</samples>
               <resolution>1</resolution>
               <min_angle>-2.35619449019</min_angle>

File: arena_robots/components/lidar/boxer_rear/lidar.urdf.xacro (robot description, xacro)
@@ -31,17 +31,17 @@
         <pose>0 0 0 0 0 0</pose>
         <visualize>false</visualize>
-        <update_rate>33</update_rate>
+        <update_rate>50</update_rate>
         <ray>
           <scan>
             <horizontal>
-              <samples>90</samples>
+              <samples>11</samples>
               <resolution>1</resolution>
-              <min_angle>0.785398163397</min_angle>
-              <max_angle>-0.785398163397</max_angle>
+              <min_angle>-0.6981317</min_angle>
+              <max_angle>0.6981317</max_angle>
             </horizontal>
           </scan>
           <range>
-            <min>0.1</min>
-            <max>5</max>
+            <min>0.2</min>
+            <max>8</max>
             <resolution>0.01</resolution>
           </range>

File: arena_robots/tests/golden/boxer_default.urdf (robot description, URDF)
Before this commit: robot boxer, 38 links, 37 joints
Joints:
- joint front_laser_joint: origin xyz=0.3062 0 0.1614 rpy=0 0 0 -> xyz=0.3062 0.0 0.1614 rpy=0.0 0.0 0.0
- joint front_realsense_mount_link_joint: origin xyz=0.3524 0 0.0422 rpy=0 -0.257610597594 0 -> xyz=0.3524 0.0 0.0422 rpy=0.0 -0.257610597594 0.0
- joint imu_sensor_link_joint: origin xyz=0 0 0 rpy=0 0 0 -> xyz=0.0 0.0 0.0 rpy=0.0 0.0 0.0
- joint rear_sensor_joint: origin xyz=-0.3404 0.0241 0.0779 rpy=0 -0.0698131700798 3.141592653589793 -> xyz=-0.3404 0.0241 0.0779 rpy=0.0 -0.0698131700798 3.141592653589793
