Commit message: robosense helios 16p mirrors the datasheet

File: arena_robots/components/lidar/robosense_helios_16p/robosense_helios_16p.urdf.xacro (robot description, xacro)
@@ -54,10 +54,11 @@
       gazebo_classic="${gazebo_classic}"
       gazebo_ignition="${gazebo_ignition}"
-      min_range="0.1"
-      max_range="50.0"
-      max_angle="85"
+      min_range="0.2"
+      max_range="150.0"
+      min_angle="-15"
+      max_angle="15"
       frame_link="${frame_prefix}link"
       rate="10"
-      horizontal_samples="1200"
+      horizontal_samples="1800"
       vertical_samples="16"
     >

File: arena_robots/components/plugins/lidar/lidar_3d_plugin.urdf.xacro (robot description, xacro)
@@ -32,5 +32,5 @@
                 <samples>${vertical_samples}</samples>
                 <resolution>1.0</resolution>
-                <min_angle>0.0</min_angle>
+                <min_angle>${radians(min_angle)}</min_angle>
                 <max_angle>${radians(max_angle)}</max_angle>
               </vertical>

File: arena_robots/tests/golden/rbsummit_default.urdf (robot description, URDF)
Before this commit: robot summit_xl, 23 links, 22 joints
Links:
- link robot_front_rgbd_camera_link: mass 0.1 -> 0.072; geometry collision box size=0.02505 0.09 0.025; visual mesh filename=package://realsense2_description/meshes/d435.dae
- link robot_top_3d_laser_base_link: geometry collision mesh filename=package://arena_robots/components/lidar/robosense_helios_16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; visual mesh filename=package://arena_robots/components/lidar/robosense_helios_16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
- link robot_vectornav_base_link: geometry collision box size=0.036 0.037 0.009; visual mesh filename=package://arena_robots/components/imu/vectornav/meshes/vect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
Joints:
- joint robot_front_rgbd_camera_joint: origin xyz=0.324 0.012 0.172 rpy=0 0 0 -> xyz=0.324 0.012 0.172 rpy=0.0 0.0 0.0
- joint robot_front_rgbd_camera_link_joint: origin xyz=0.0106 0.0175 0.0125 rpy=0 0 0 -> xyz=0.010600000000000002 0.0175 0.0125 rpy=0 0 0
- joint robot_top_3d_laser_base_joint: origin xyz=-0.01924 0.0 0.27642 rpy=0 0 0 -> xyz=-0.01924 0.0 0.27642 rpy=0.0 0.0 0.0
- joint robot_vectornav_base_joint: origin xyz=0.0385 0.132 0.158 rpy=0 0 0 -> xyz=0.0385 0.132 0.158 rpy=0.0 0.0 0.0
