Commit message: sick microscan3 mirrors the datasheet

File: arena_robots/components/lidar/sick_microscan3/sick_microscan3.urdf.xacro (robot description, xacro)
@@ -55,10 +55,10 @@
       min_range="0.05"
       max_range="64.0"
-      min_angle="-2.35"
-      max_angle="2.35"
+      min_angle="-2.39982772"
+      max_angle="2.39982772"
       frame_link="${frame_prefix}link"
-      rate="30"
+      rate="33"
       resolution="0.00575"
-      samples="700"
+      samples="2751"
     >
     </xacro:lidar_2d_plugin>

File: arena_robots/tests/golden/rbrobout_default.urdf (robot description, URDF)
Before this commit: robot rbrobout, 16 links, 15 joints
Links:
- link robot_front_laser_base_link: geometry collision mesh filename=package://arena_robots/components/lidar/sick_microscan3/mes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; visual mesh filename=package://arena_robots/components/lidar/sick_microscan3/mes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
- link robot_rear_laser_base_link: geometry collision mesh filename=package://arena_robots/components/lidar/sick_microscan3/mes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; visual mesh filename=package://arena_robots/components/lidar/sick_microscan3/mes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
- link robot_vectornav_base_link: geometry collision box size=0.036 0.037 0.009; visual mesh filename=package://arena_robots/components/imu/vectornav/meshes/vect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
Joints:
- joint robot_front_laser_base_joint: origin xyz=0.8 0.366 -0.06 rpy=0 0 0.7853981633975 -> xyz=0.8 0.366 -0.06 rpy=0.0 0.0 0.7853981633974483
- joint robot_rear_laser_base_joint: origin xyz=-0.8 -0.366 -0.06 rpy=0 0 -2.3561944901925003 -> xyz=-0.8 -0.366 -0.06 rpy=0.0 0.0 -2.356194490192345
- joint robot_vectornav_base_joint: origin xyz=0.3 -0.3 0.0725 rpy=0 0 0 -> xyz=0.3 -0.3 0.0725 rpy=0.0 0.0 0.0
